Commit message: Add full bin xacro file and friction coefficients

File: amrj16_bin_description/urdf/amrj16_full_bin.xacro (robot description, xacro)
@@ -1,6 +1,6 @@
 <?xml version="1.0"?>
-<robot xmlns:xacro="http://www.ros.org/wiki/xacro" name="empty_bin">
+<robot xmlns:xacro="http://www.ros.org/wiki/xacro" name="full_bin">
     <!-- Definizione della variabile prefix -->
-    <xacro:property name="prefix" value="empty_bin"/>
+    <xacro:property name="prefix" value="full_bin"/>
     <!-- Link e giunti con prefix -->
     <link name="${prefix}_base_footprint">
@@ -53,5 +53,5 @@
         </collision>
         <inertial>
-            <mass value="0.7"/>
+            <mass value="0.5"/>
             <origin rpy="0 0 0" xyz="0 0 0"/>
             <inertia ixx="0.0008063" ixy="0.00000393" ixz="-0.00000650" iyy="0.000693" iyz="0.000265" izz="0.0005498"/>
@@ -63,131 +63,9 @@
         <child link="${prefix}_front_right_caster_hub"/>
         <axis xyz="0 0 1"/>
+        <limit effort="1000.0" velocity="100.0" />
         <dynamics damping="0.5" friction="0.1"/>
     </joint>
  <!-- front-right caster wheel -->
             <link name="${prefix}_front_right_caster_wheel">
-        <visual>
-            <origin xyz="0 0 0" rpy="1.57 0 0"/>
-                <geometry>
-                    <mesh filename="package://amrj16_bin_description/models/meshes/utimac_wheel_bin_v1.dae"/>
-                </geometry>
-        </visual>
-    <collision>
-        <origin xyz="0 0 0" rpy="1.57  0 0"/>
-        <geometry>
-                <cylinder radius="0.04" length="0.02"/>
-        </geometry>
-    </collision>
-    <inertial>
-        <mass value="0.7"/>
-        <origin rpy="0 0 0" xyz="1.57  0 0"/>
-        <inertia
-            ixx="0.0003265" ixy="0" ixz="0" iyy="0.0003265" iyz="0" izz="0.0005849"/>
-    </inertial>
-    </link>
-    <gazebo reference="${prefix}_front_right_caster_wheel">
-        <kp>1000000000000000000000000000.0</kp>
-        <kd>1000000000000000000000000000.0</kd>
-        <mu1>10.0</mu1>
-        <mu2>10.0</mu2>
-    </gazebo>
-    <joint name="${prefix}_front_right_caster_hub_wheel_joint" type="continuous">
-       <origin xyz="0.039 0 -0.067" rpy="0 0 0"/>
-        <parent link="${prefix}_front_right_caster_hub"/>
-        <child link="${prefix}_front_right_caster_wheel"/>
-        <axis xyz="0 1 0"/>
-        <dynamics damping="0.5" friction="0.1"/>
-    </joint>
- <!-- front-left caster hub -->
-    <link name="${prefix}_front_left_caster_hub">
-        <visual>
-            <origin xyz="0 0 0" rpy="0 0 0"/>
-            <geometry>
-                <mesh filename="package://amrj16_bin_description/models/meshes/utimac_caster_bin_v1.dae"/>
-            </geometry>
-        </visual>
-        <collision>
-            <origin xyz="0 0 0" rpy="0 0 0"/>
-            <geometry>
-                <mesh filename="package://amrj16_bin_description/models/meshes/utimac_caster_bin_v1.dae"/>
-            </geometry>
-        </collision>
-        <inertial>
-            <mass value="0.5"/>
-            <origin rpy="0 0 0" xyz="0 0 0"/>
-            <inertia ixx="0.0008063" ixy="0.00000393" ixz="-0.00000650" iyy="0.000693" iyz="0.000265" izz="0.0005498"/>
-        </inertial>
-    </link>
-    <joint name="${prefix}_chassis_front_left_caster_hub_joint" type="continuous">
-       <origin xyz="0.2925 -0.215 0" rpy="0 0 0"/>
-        <parent link="${prefix}_chassis"/>
-        <child link="${prefix}_front_left_caster_hub"/>
-        <axis xyz="0 0 1"/>
-        <limit effort="1000.0" velocity="100.0" />
-        <dynamics damping="0.5" friction="0.1"/>
-    </joint>
-<!-- front-left caster wheel -->
-            <link name="${prefix}_front_left_caster_wheel">
-        <visual>
-            <origin xyz="0 0 0" rpy="1.57 0 0"/>
-                <geometry>
-                    <mesh filename="package://amrj16_bin_description/models/meshes/utimac_wheel_bin_v1.dae"/>
-                </geometry>
-        </visual>
-    <collision>
-        <origin xyz="0 0 0" rpy="1.57  0 0"/>
-        <geometry>
-                <cylinder radius="0.04" length="0.02"/>
-        </geometry>
-    </collision>
-    <inertial>
-        <mass value="0.7"/>
-        <origin rpy="0 0 0" xyz="1.57  0 0"/>
-        <inertia
-            ixx="0.0003265" ixy="0" ixz="0" iyy="0.0003265" iyz="0" izz="0.0005849"/>
-    </inertial>
-    </link>
-    <gazebo reference="${prefix}_front_left_caster_wheel">
-        <kp>1000000000000000000000000000.0</kp>
-        <kd>1000000000000000000000000000.0</kd>
-        <mu1>10.0</mu1>
-        <mu2>10.0</mu2>
-    </gazebo>
-    <joint name="${prefix}_front_left_caster_hub_wheel_joint" type="continuous">
-       <origin xyz="0.039 0 -0.067" rpy="0 0 0"/>
-        <parent link="${prefix}_front_left_caster_hub"/>
-        <child link="${prefix}_front_left_caster_wheel"/>
-        <axis xyz="0 1 0"/>
-        <dynamics damping="0.5" friction="0.1"/>
-    </joint>
-  <!-- rear-right caster hub -->
-    <link name="${prefix}_rear_right_caster_hub">
-        <visual>
-            <origin xyz="0 0 0" rpy="0 0 0"/>
-            <geometry>
-                <mesh filename="package://amrj16_bin_description/models/meshes/utimac_caster_bin_v1.dae"/>
-            </geometry>
-        </visual>
-        <collision>
-            <origin xyz="0 0 0" rpy="0 0 0"/>
-            <geometry>
-                <mesh filename="package://amrj16_bin_description/models/meshes/utimac_caster_bin_v1.dae"/>
-            </geometry>
-        </collision>
-        <inertial>
-            <mass value="0.7"/>
-            <origin rpy="0 0 0" xyz="0 0 0"/>
-            <inertia ixx="0.0008063" ixy="0.00000393" ixz="-0.00000650" iyy="0.000693" iyz="0.000265" izz="0.0005498"/>
-        </inertial>
-    </link>
-    <joint name="${prefix}_chassis_rear_right_caster_hub_joint" type="continuous">
-       <origin xyz="-0.2925 0.215 0" rpy="0 0 0"/>
-        <parent link="${prefix}_chassis"/>
-        <child link="${prefix}_rear_right_caster_hub"/>
-        <axis xyz="0 0 1"/>
-        <dynamics damping="0.5" friction="0.1"/>
-    </joint>
- <!-- rear-right caster wheel -->
-            <link name="${prefix}_rear_right_caster_wheel">
         <visual>
             <origin xyz="0 0 0" rpy="1.57 0 0"/>
@@ -209,5 +87,5 @@
     </inertial>
     </link>
-   <gazebo reference="${prefix}_rear_right_caster_wheel">
+    <gazebo reference="${prefix}_front_right_caster_wheel">
         <kp>1000000000000000000000000000.0</kp>
         <kd>1000000000000000000000000000.0</kd>
@@ -215,13 +93,14 @@
         <mu2>10.0</mu2>
     </gazebo>
-    <joint name="${prefix}_rear_right_caster_hub_wheel_joint" type="continuous">
+    <joint name="${prefix}_front_right_caster_hub_wheel_joint" type="continuous">
        <origin xyz="0.039 0 -0.067" rpy="0 0 0"/>
-        <parent link="${prefix}_rear_right_caster_hub"/>
-        <child link="${prefix}_rear_right_caster_wheel"/>
+        <parent link="${prefix}_front_right_caster_hub"/>
+        <child link="${prefix}_front_right_caster_wheel"/>
         <axis xyz="0 1 0"/>
-        <dynamics damping="0.5" friction="0.1"/>
-    </joint>
-<!-- rear-left caster hub -->
-    <link name="${prefix}_rear_left_caster_hub">
+        <limit effort="1000.0" velocity="100.0" />
+        <dynamics damping="0.5" friction="0.1"/>
+    </joint>
+ <!-- front-left caster hub -->
+    <link name="${prefix}_front_left_caster_hub">
         <visual>
             <origin xyz="0 0 0" rpy="0 0 0"/>
@@ -242,13 +121,14 @@
         </inertial>
     </link>
-    <joint name="${prefix}_chassis_rear_left_caster_hub_joint" type="continuous">
-       <origin xyz="-0.2925 -0.215 0" rpy="0 0 0"/>
+    <joint name="${prefix}_chassis_front_left_caster_hub_joint" type="continuous">
+       <origin xyz="0.2925 -0.215 0" rpy="0 0 0"/>
         <parent link="${prefix}_chassis"/>
-        <child link="${prefix}_rear_left_caster_hub"/>
+        <child link="${prefix}_front_left_caster_hub"/>
         <axis xyz="0 0 1"/>
-        <dynamics damping="0.5" friction="0.1"/>
-    </joint>
-<!-- rear-left caster wheel -->
-            <link name="${prefix}_rear_left_caster_wheel">
+        <limit effort="1000.0" velocity="100.0" />
+        <dynamics damping="0.5" friction="0.1"/>
+    </joint>
+<!-- front-left caster wheel -->
+            <link name="${prefix}_front_left_caster_wheel">
         <visual>
             <origin xyz="0 0 0" rpy="1.57 0 0"/>
@@ -264,5 +144,131 @@
     </collision>
     <inertial>
-        <mass value="0.5"/>
+        <mass value="0.8"/>
+        <origin rpy="0 0 0" xyz="1.57  0 0"/>
+        <inertia
+            ixx="0.0003265" ixy="0" ixz="0" iyy="0.0003265" iyz="0" izz="0.0005849"/>
+    </inertial>
+    </link>
+    <gazebo reference="${prefix}_front_left_caster_wheel">
+        <kp>1000000000000000000000000000.0</kp>
+        <kd>1000000000000000000000000000.0</kd>
+        <mu1>10.0</mu1>
+        <mu2>10.0</mu2>
+    </gazebo>
+    <joint name="${prefix}_front_left_caster_hub_wheel_joint" type="continuous">
+       <origin xyz="0.039 0 -0.067" rpy="0 0 0"/>
+        <parent link="${prefix}_front_left_caster_hub"/>
+        <child link="${prefix}_front_left_caster_wheel"/>
+        <axis xyz="0 1 0"/>
+        <limit effort="1000.0" velocity="100.0" />
+        <dynamics damping="0.5" friction="0.1"/>
+    </joint>
+  <!-- rear-right caster hub -->
+    <link name="${prefix}_rear_right_caster_hub">
+        <visual>
+            <origin xyz="0 0 0" rpy="0 0 0"/>
+            <geometry>
+                <mesh filename="package://amrj16_bin_description/models/meshes/utimac_caster_bin_v1.dae"/>
+            </geometry>
+        </visual>
+        <collision>
+            <origin xyz="0 0 0" rpy="0 0 0"/>
+            <geometry>
+                <mesh filename="package://amrj16_bin_description/models/meshes/utimac_caster_bin_v1.dae"/>
+            </geometry>
+        </collision>
+        <inertial>
+            <mass value="0.5"/>
+            <origin rpy="0 0 0" xyz="0 0 0"/>
+            <inertia ixx="0.0008063" ixy="0.00000393" ixz="-0.00000650" iyy="0.000693" iyz="0.000265" izz="0.0005498"/>
+        </inertial>
+    </link>
+    <joint name="${prefix}_chassis_rear_right_caster_hub_joint" type="continuous">
+       <origin xyz="-0.2925 0.215 0" rpy="0 0 0"/>
+        <parent link="${prefix}_chassis"/>
+        <child link="${prefix}_rear_right_caster_hub"/>
+        <axis xyz="0 0 1"/>
+        <limit effort="1000.0" velocity="100.0" />
+        <dynamics damping="0.5" friction="0.1"/>
+    </joint>
+ <!-- rear-right caster wheel -->
+            <link name="${prefix}_rear_right_caster_wheel">
+        <visual>
+            <origin xyz="0 0 0" rpy="1.57 0 0"/>
+                <geometry>
+                    <mesh filename="package://amrj16_bin_description/models/meshes/utimac_wheel_bin_v1.dae"/>
+                </geometry>
+        </visual>
+    <collision>
+        <origin xyz="0 0 0" rpy="1.57  0 0"/>
+        <geometry>
+                <cylinder radius="0.04" length="0.02"/>
+        </geometry>
+    </collision>
+    <inertial>
+        <mass value="0.8"/>
+        <origin rpy="0 0 0" xyz="1.57  0 0"/>
+        <inertia
+            ixx="0.0003265" ixy="0" ixz="0" iyy="0.0003265" iyz="0" izz="0.0005849"/>
+    </inertial>
+    </link>
+   <gazebo reference="${prefix}_rear_right_caster_wheel">
+        <kp>1000000000000000000000000000.0</kp>
+        <kd>1000000000000000000000000000.0</kd>
+        <mu1>10.0</mu1>
+        <mu2>10.0</mu2>
+    </gazebo>
+    <joint name="${prefix}_rear_right_caster_hub_wheel_joint" type="continuous">
+       <origin xyz="0.039 0 -0.067" rpy="0 0 0"/>
+        <parent link="${prefix}_rear_right_caster_hub"/>
+        <child link="${prefix}_rear_right_caster_wheel"/>
+        <axis xyz="0 1 0"/>
+        <limit effort="1000.0" velocity="100.0" />
+        <dynamics damping="0.5" friction="0.1"/>
+    </joint>
+<!-- rear-left caster hub -->
+    <link name="${prefix}_rear_left_caster_hub">
+        <visual>
+            <origin xyz="0 0 0" rpy="0 0 0"/>
+            <geometry>
+                <mesh filename="package://amrj16_bin_description/models/meshes/utimac_caster_bin_v1.dae"/>
+            </geometry>
+        </visual>
+        <collision>
+            <origin xyz="0 0 0" rpy="0 0 0"/>
+            <geometry>
+                <mesh filename="package://amrj16_bin_description/models/meshes/utimac_caster_bin_v1.dae"/>
+            </geometry>
+        </collision>
+        <inertial>
+            <mass value="0.5"/>
+            <origin rpy="0 0 0" xyz="0 0 0"/>
+            <inertia ixx="0.0008063" ixy="0.00000393" ixz="-0.00000650" iyy="0.000693" iyz="0.000265" izz="0.0005498"/>
+        </inertial>
+    </link>
+    <joint name="${prefix}_chassis_rear_left_caster_hub_joint" type="continuous">
+       <origin xyz="-0.2925 -0.215 0" rpy="0 0 0"/>
+        <parent link="${prefix}_chassis"/>
+        <child link="${prefix}_rear_left_caster_hub"/>
+        <axis xyz="0 0 1"/>
+        <limit effort="1000.0" velocity="100.0" />
+        <dynamics damping="0.5" friction="0.1"/>
+    </joint>
+<!-- rear-left caster wheel -->
+            <link name="${prefix}_rear_left_caster_wheel">
+        <visual>
+            <origin xyz="0 0 0" rpy="1.57 0 0"/>
+                <geometry>
+                    <mesh filename="package://amrj16_bin_description/models/meshes/utimac_wheel_bin_v1.dae"/>
+                </geometry>
+        </visual>
+    <collision>
+        <origin xyz="0 0 0" rpy="1.57  0 0"/>
+        <geometry>
+                <cylinder radius="0.04" length="0.02"/>
+        </geometry>
+    </collision>
+    <inertial>
+        <mass value="0.8"/>
         <origin rpy="0 0 0" xyz="1.57  0 0"/>
         <inertia

Commit message: Updating the environment and coefficients to strengthen stability

File: amrj16_bin_description/urdf/amrj16_full_bin.xacro (robot description, xacro)
@@ -22,12 +22,12 @@
         </visual>
         <collision>
-            <origin xyz="0 0 0" rpy="0 0 0"/>
-            <geometry>
-                <mesh filename="package://amrj16_bin_description/models/meshes/utimac_bin_v1.dae"/>
+            <origin xyz="0 0 0.2" rpy="0 0 0"/>
+            <geometry>
+                <box size="0.815 0.690 0.293" />
             </geometry>
         </collision>
         <inertial>
             <mass value="38"/>
-            <origin rpy="0 0 0" xyz="0 0 0"/>
+            <origin  xyz="0 0 0" rpy="0 0 0"/>
             <inertia ixx="8.1" ixy="0.00213" ixz="4.56" iyy="11.5" iyz="-0.00156" izz="7.71"/>
         </inertial>
@@ -46,12 +46,12 @@
             </geometry>
         </visual>
-        <collision>
-            <origin xyz="0 0 0" rpy="0 0 0"/>
-            <geometry>
-                <mesh filename="package://amrj16_bin_description/models/meshes/utimac_caster_bin_v1.dae"/>
-            </geometry>
-        </collision>
-        <inertial>
-            <mass value="0.5"/>
+        <!--collision>
+            <origin xyz="0 0 0" rpy="0 0 0"/>
+            <geometry>
+                <mesh filename="package://amrj16_bin_description/models/meshes/utimac_caster_bin_v1.dae"/>
+            </geometry>
+        </collision -->
+        <inertial>
+            <mass value="1"/>
             <origin rpy="0 0 0" xyz="0 0 0"/>
             <inertia ixx="0.0008063" ixy="0.00000393" ixz="-0.00000650" iyy="0.000693" iyz="0.000265" izz="0.0005498"/>
@@ -63,6 +63,5 @@
         <child link="${prefix}_front_right_caster_hub"/>
         <axis xyz="0 0 1"/>
-        <limit effort="1000.0" velocity="100.0" />
-        <dynamics damping="0.5" friction="0.1"/>
+              <dynamics damping="0.5" friction="0.1"/>
     </joint>
  <!-- front-right caster wheel -->
@@ -81,5 +80,5 @@
     </collision>
     <inertial>
-        <mass value="0.5"/>
+        <mass value="1"/>
         <origin rpy="0 0 0" xyz="1.57  0 0"/>
         <inertia
@@ -88,6 +87,6 @@
     </link>
     <gazebo reference="${prefix}_front_right_caster_wheel">
-        <kp>1000000000000000000000000000.0</kp>
-        <kd>1000000000000000000000000000.0</kd>
+        <kp>1e6</kp>
+        <kd>1e3</kd>
         <mu1>10.0</mu1>
         <mu2>10.0</mu2>
@@ -98,6 +97,5 @@
         <child link="${prefix}_front_right_caster_wheel"/>
         <axis xyz="0 1 0"/>
-        <limit effort="1000.0" velocity="100.0" />
-        <dynamics damping="0.5" friction="0.1"/>
+        <dynamics damping="0.5" friction="0.5"/>
     </joint>
  <!-- front-left caster hub -->
@@ -109,12 +107,12 @@
             </geometry>
         </visual>
-        <collision>
-            <origin xyz="0 0 0" rpy="0 0 0"/>
-            <geometry>
-                <mesh filename="package://amrj16_bin_description/models/meshes/utimac_caster_bin_v1.dae"/>
-            </geometry>
-        </collision>
-        <inertial>
-            <mass value="0.5"/>
+        <!--collision>
+            <origin xyz="0 0 0" rpy="0 0 0"/>
+            <geometry>
+                <mesh filename="package://amrj16_bin_description/models/meshes/utimac_caster_bin_v1.dae"/>
+            </geometry>
+        </collision -->
+        <inertial>
+            <mass value="1"/>
             <origin rpy="0 0 0" xyz="0 0 0"/>
             <inertia ixx="0.0008063" ixy="0.00000393" ixz="-0.00000650" iyy="0.000693" iyz="0.000265" izz="0.0005498"/>
@@ -126,5 +124,4 @@
         <child link="${prefix}_front_left_caster_hub"/>
         <axis xyz="0 0 1"/>
-        <limit effort="1000.0" velocity="100.0" />
         <dynamics damping="0.5" friction="0.1"/>
     </joint>
@@ -144,5 +141,5 @@
     </collision>
     <inertial>
-        <mass value="0.8"/>
+        <mass value="1"/>
         <origin rpy="0 0 0" xyz="1.57  0 0"/>
         <inertia
@@ -151,6 +148,6 @@
     </link>
     <gazebo reference="${prefix}_front_left_caster_wheel">
-        <kp>1000000000000000000000000000.0</kp>
-        <kd>1000000000000000000000000000.0</kd>
+        <kp>1e6</kp>
+        <kd>1e3</kd>
         <mu1>10.0</mu1>
         <mu2>10.0</mu2>
@@ -161,6 +158,5 @@
         <child link="${prefix}_front_left_caster_wheel"/>
         <axis xyz="0 1 0"/>
-        <limit effort="1000.0" velocity="100.0" />
-        <dynamics damping="0.5" friction="0.1"/>
+        <dynamics damping="0.5" friction="0.5"/>
     </joint>
   <!-- rear-right caster hub -->
@@ -172,12 +168,12 @@
             </geometry>
         </visual>
-        <collision>
-            <origin xyz="0 0 0" rpy="0 0 0"/>
-            <geometry>
-                <mesh filename="package://amrj16_bin_description/models/meshes/utimac_caster_bin_v1.dae"/>
-            </geometry>
-        </collision>
-        <inertial>
-            <mass value="0.5"/>
+        <!--collision>
+            <origin xyz="0 0 0" rpy="0 0 0"/>
+            <geometry>
+                <mesh filename="package://amrj16_bin_description/models/meshes/utimac_caster_bin_v1.dae"/>
+            </geometry>
+        </collision -->
+        <inertial>
+            <mass value="1"/>
             <origin rpy="0 0 0" xyz="0 0 0"/>
             <inertia ixx="0.0008063" ixy="0.00000393" ixz="-0.00000650" iyy="0.000693" iyz="0.000265" izz="0.0005498"/>
@@ -189,5 +185,4 @@
         <child link="${prefix}_rear_right_caster_hub"/>
         <axis xyz="0 0 1"/>
-        <limit effort="1000.0" velocity="100.0" />
         <dynamics damping="0.5" friction="0.1"/>
     </joint>
@@ -207,5 +202,5 @@
     </collision>
     <inertial>
-        <mass value="0.8"/>
+        <mass value="1"/>
         <origin rpy="0 0 0" xyz="1.57  0 0"/>
         <inertia
@@ -214,6 +209,6 @@
     </link>
    <gazebo reference="${prefix}_rear_right_caster_wheel">
-        <kp>1000000000000000000000000000.0</kp>
-        <kd>1000000000000000000000000000.0</kd>
+        <kp>1e6</kp>
+        <kd>1e3</kd>
         <mu1>10.0</mu1>
         <mu2>10.0</mu2>
@@ -224,6 +219,5 @@
         <child link="${prefix}_rear_right_caster_wheel"/>
         <axis xyz="0 1 0"/>
-        <limit effort="1000.0" velocity="100.0" />
-        <dynamics damping="0.5" friction="0.1"/>
+        <dynamics damping="0.5" friction="0.5"/>
     </joint>
 <!-- rear-left caster hub -->
@@ -235,12 +229,12 @@
             </geometry>
         </visual>
-        <collision>
-            <origin xyz="0 0 0" rpy="0 0 0"/>
-            <geometry>
-                <mesh filename="package://amrj16_bin_description/models/meshes/utimac_caster_bin_v1.dae"/>
-            </geometry>
-        </collision>
-        <inertial>
-            <mass value="0.5"/>
+        <!--collision>
+            <origin xyz="0 0 0" rpy="0 0 0"/>
+            <geometry>
+                <mesh filename="package://amrj16_bin_description/models/meshes/utimac_caster_bin_v1.dae"/>
+            </geometry>
+        </collision -->
+        <inertial>
+            <mass value="1"/>
             <origin rpy="0 0 0" xyz="0 0 0"/>
             <inertia ixx="0.0008063" ixy="0.00000393" ixz="-0.00000650" iyy="0.000693" iyz="0.000265" izz="0.0005498"/>
@@ -252,5 +246,4 @@
         <child link="${prefix}_rear_left_caster_hub"/>
         <axis xyz="0 0 1"/>
-        <limit effort="1000.0" velocity="100.0" />
         <dynamics damping="0.5" friction="0.1"/>
     </joint>
@@ -270,5 +263,5 @@
     </collision>
     <inertial>
-        <mass value="0.8"/>
+        <mass value="1"/>
         <origin rpy="0 0 0" xyz="1.57  0 0"/>
         <inertia
@@ -277,6 +270,6 @@
     </link>
     <gazebo reference="${prefix}_rear_left_caster_wheel">
-        <kp>1000000000000000000000000000.0</kp>
-        <kd>1000000000000000000000000000.0</kd>
+        <kp>1e6</kp>
+        <kd>1e3</kd>
         <mu1>10.0</mu1>
         <mu2>10.0</mu2>
@@ -287,5 +280,5 @@
         <child link="${prefix}_rear_left_caster_wheel"/>
         <axis xyz="0 1 0"/>
-        <dynamics damping="0.5" friction="0.1"/>
+        <dynamics damping="0.5" friction="0.5"/>
     </joint>
     <!-- Plugin Gazebo -->
