Commit message: Troubleshooting laser and navigation problems

File: amrj16_bin_description/urdf/amrj16_full_bin.xacro (robot description, xacro)
@@ -87,8 +87,19 @@
     </link>
     <gazebo reference="${prefix}_front_right_caster_wheel">
-        <kp>1e6</kp>
-        <kd>1e3</kd>
-        <mu1>10.0</mu1>
-        <mu2>10.0</mu2>
+      <collision>
+        <surface>
+          <friction>
+            <ode>
+              <mu>0.3</mu>
+              <mu2>0.3</mu2>
+            </ode>
+            <bullet>
+              <friction>0.3</friction>
+              <friction2>0.3</friction2>
+              <rolling_friction>0.1</rolling_friction>
+            </bullet>
+          </friction>
+        </surface>
+      </collision>
     </gazebo>
     <joint name="${prefix}_front_right_caster_hub_wheel_joint" type="continuous">
@@ -97,5 +108,5 @@
         <child link="${prefix}_front_right_caster_wheel"/>
         <axis xyz="0 1 0"/>
-        <dynamics damping="0.5" friction="0.5"/>
+        <dynamics damping="0.5" friction="1.5"/>
     </joint>
  <!-- front-left caster hub -->
@@ -148,8 +159,19 @@
     </link>
     <gazebo reference="${prefix}_front_left_caster_wheel">
-        <kp>1e6</kp>
-        <kd>1e3</kd>
-        <mu1>10.0</mu1>
-        <mu2>10.0</mu2>
+      <collision>
+        <surface>
+          <friction>
+            <ode>
+              <mu>0.3</mu>
+              <mu2>0.3</mu2>
+            </ode>
+            <bullet>
+              <friction>0.3</friction>
+              <friction2>0.3</friction2>
+              <rolling_friction>0.1</rolling_friction>
+            </bullet>
+          </friction>
+        </surface>
+      </collision>
     </gazebo>
     <joint name="${prefix}_front_left_caster_hub_wheel_joint" type="continuous">
@@ -158,5 +180,5 @@
         <child link="${prefix}_front_left_caster_wheel"/>
         <axis xyz="0 1 0"/>
-        <dynamics damping="0.5" friction="0.5"/>
+        <dynamics damping="0.5" friction="1.5"/>
     </joint>
   <!-- rear-right caster hub -->
@@ -209,8 +231,19 @@
     </link>
    <gazebo reference="${prefix}_rear_right_caster_wheel">
-        <kp>1e6</kp>
-        <kd>1e3</kd>
-        <mu1>10.0</mu1>
-        <mu2>10.0</mu2>
+      <collision>
+        <surface>
+          <friction>
+            <ode>
+              <mu>0.3</mu>
+              <mu2>0.3</mu2>
+            </ode>
+            <bullet>
+              <friction>0.3</friction>
+              <friction2>0.3</friction2>
+              <rolling_friction>0.1</rolling_friction>
+            </bullet>
+          </friction>
+        </surface>
+      </collision>
     </gazebo>
     <joint name="${prefix}_rear_right_caster_hub_wheel_joint" type="continuous">
@@ -219,5 +252,5 @@
         <child link="${prefix}_rear_right_caster_wheel"/>
         <axis xyz="0 1 0"/>
-        <dynamics damping="0.5" friction="0.5"/>
+        <dynamics damping="0.5" friction="1.5"/>
     </joint>
 <!-- rear-left caster hub -->
@@ -270,8 +303,19 @@
     </link>
     <gazebo reference="${prefix}_rear_left_caster_wheel">
-        <kp>1e6</kp>
-        <kd>1e3</kd>
-        <mu1>10.0</mu1>
-        <mu2>10.0</mu2>
+      <collision>
+        <surface>
+          <friction>
+            <ode>
+              <mu>0.3</mu>
+              <mu2>0.3</mu2>
+            </ode>
+            <bullet>
+              <friction>0.3</friction>
+              <friction2>0.3</friction2>
+              <rolling_friction>0.1</rolling_friction>
+            </bullet>
+          </friction>
+        </surface>
+      </collision>
     </gazebo>
     <joint name="${prefix}_rear_left_caster_hub_wheel_joint" type="continuous">
@@ -280,5 +324,5 @@
         <child link="${prefix}_rear_left_caster_wheel"/>
         <axis xyz="0 1 0"/>
-        <dynamics damping="0.5" friction="0.5"/>
+        <dynamics damping="0.5" friction="1.5"/>
     </joint>
     <!-- Plugin Gazebo -->

File: amrj16_description/urdf/amrj16.xacro (robot description, xacro)
@@ -15,5 +15,5 @@
       <origin xyz="0 0 0" rpy="0 0 0"/>
       <geometry>
-        <mesh filename="package://amrj16_description/models/meshes/amrj16_chassis_utimac_v1.dae"/>
+        <mesh filename="package://amrj16_description/models/meshes/amrj16_chassis_utimac_v2.dae"/>
       </geometry>
     </visual>
@@ -21,5 +21,5 @@
       <origin xyz="0 0 0" rpy="0 0 0"/>
       <geometry>
-        <mesh filename="package://amrj16_description/models/meshes/amrj16_chassis_utimac_v1.dae"/>
+        <mesh filename="package://amrj16_description/models/meshes/amrj16_chassis_utimac_v2_low_res.stl"/>
       </geometry>
     </collision>
@@ -62,5 +62,5 @@
     </gazebo>
     <joint name="chassis_right_wheel_joint" type="continuous">
-        <origin xyz="0 0.5456 0" rpy="1.5707 0 0"/>
+        <origin xyz="0 -0.5456 0" rpy="-1.5707 0 0"/>
         <parent link="chassis"/>
         <child link="right_wheel"/>
@@ -97,5 +97,5 @@
     </gazebo>
     <joint name="chassis_left_wheel_joint" type="continuous">
-        <origin xyz="0 -0.5456 0" rpy="1.5707 0 0"/>
+        <origin xyz="0 0.5456 0" rpy="-1.5707 0 0"/>
         <parent link="chassis"/>
         <child link="left_wheel"/>
@@ -112,10 +112,10 @@
                 </geometry>
         </visual>
-    <collision>
+    <!--collision>
         <origin xyz="0 0 0" rpy="0 0 0"/>
         <geometry>
                  <mesh filename="package://amrj16_description/models/meshes/amrj16_caster_hub.dae"/>
         </geometry>
-    </collision>
+    </collision-->
     <inertial>
         <mass value="0.140"/>
@@ -126,9 +126,8 @@
     </link>
     <joint name="chassis_front_right_caster_hub_joint" type="continuous">
-        <origin xyz="0.255 0.186 -0.05" rpy="0 0 1.5707"/>
+        <origin xyz="-0.255 -0.186 -0.05" rpy="0 0 1.5707"/>
         <parent link="chassis"/>
         <child link="front_right_caster_hub"/>
         <axis xyz="0 0 1"/>
-        <limit effort="1000.0" velocity="100.0" />
         <dynamics damping="0.0" friction="0.1"/>
     </joint>
@@ -144,5 +143,5 @@
         <origin xyz="0 0 0" rpy="0 0 0"/>
         <geometry>
-                 <mesh filename="package://amrj16_description/models/meshes/amrj16_caster_wheel.dae"/>
+            <cylinder radius="0.015" length="0.02"/>
         </geometry>
     </collision>
@@ -155,6 +154,6 @@
     </link>
     <gazebo reference="front_right_caster_wheel">
-        <kp>1000000000000000000000000000.0</kp>
-        <kd>1000000000000000000000000000.0</kd>
+        <kp>500</kp>
+        <kd>500</kd>
         <mu1>10.0</mu1>
         <mu2>10.0</mu2>
@@ -176,10 +175,10 @@
                 </geometry>
         </visual>
-        <collision>
+        <!--collision>
             <origin xyz="0 0 0" rpy="0 0 0"/>
             <geometry>
                     <mesh filename="package://amrj16_description/models/meshes/amrj16_caster_hub.dae"/>
             </geometry>
-        </collision>
+        </collision-->
         <inertial>
             <mass value="0.140"/>
@@ -190,9 +189,8 @@
     </link>
     <joint name="chassis_front_left_caster_hub_joint" type="continuous">
-        <origin xyz="0.255 -0.186 -0.05" rpy="0 0 1.5707"/>
+        <origin xyz="-0.255 0.186 -0.05" rpy="0 0 1.5707"/>
         <parent link="chassis"/>
         <child link="front_left_caster_hub"/>
         <axis xyz="0 0 1"/>
-        <limit effort="1000.0" velocity="100.0" />
         <dynamics damping="0.0" friction="0.1"/>
     </joint>
@@ -208,5 +206,5 @@
             <origin xyz="0 0 0" rpy="0 0 0"/>
             <geometry>
-                   <mesh filename="package://amrj16_description/models/meshes/amrj16_caster_wheel.dae"/>
+                <cylinder radius="0.015" length="0.02"/>
             </geometry>
         </collision>
@@ -219,6 +217,6 @@
     </link>
     <gazebo reference="front_left_caster_wheel">
-        <kp>1000000000000000000000000000.0</kp>
-        <kd>1000000000000000000000000000.0</kd>
+        <kp>500</kp>
+        <kd>500</kd>
         <mu1>10.0</mu1>
         <mu2>10.0</mu2>
@@ -236,5 +234,5 @@
     </link>
     <joint name="camera_dx_joint" type="fixed">
-        <origin rpy="0 0 0" xyz="0.280 0.186 -0.035"/>
+        <origin rpy="0 0 0" xyz="-0.280 -0.186 -0.035"/>
         <parent link="chassis" />
         <child link="rgb_camera_dx" />
@@ -280,5 +278,5 @@
     </link>
     <joint name="rgb_camera_sx_joint" type="fixed">
-        <origin rpy="0 0 0" xyz="0.280 -0.186 -0.035"/>
+        <origin rpy="0 0 0" xyz="-0.280 0.186 -0.035"/>
         <parent link="chassis" />
         <child link="rgb_camera_sx" />
@@ -342,5 +340,5 @@
     </link>
     <joint name="chassis_lidar_joint" type="fixed">
-        <origin rpy="0 0 0" xyz="0.200 0 -0.06"/>
+        <origin rpy="0 0 3.14" xyz="-0.2 0 0.2"/>
         <parent link="chassis" />
         <child link="lidar" />
@@ -380,5 +378,5 @@
     </link>
     <joint name="chassis_asus_xtion_joint" type="fixed">
-        <origin rpy="0 0 0" xyz="0.300 0.0 0.2465"/>
+        <origin rpy="0 0 0" xyz="0.300 0.0 0.2"/>
         <parent link="chassis" />
         <child link="asus_xtion" />
@@ -516,15 +514,16 @@
       <wheel_diameter>0.206</wheel_diameter>
       <!-- limits -->
-      <max_wheel_torque>1.0</max_wheel_torque>
-      <max_wheel_acceleration>1.0</max_wheel_acceleration>
-      <!--command_topic>cmd_vel</command_topic -->
+      <max_wheel_torque>20.0</max_wheel_torque>
+      <max_wheel_acceleration>0.3</max_wheel_acceleration>
+      <command_topic>cmd_vel</command_topic>
       <!-- remapping>/cmd_vel:=/cmd_vel</remapping -->
       <!-- output -->
       <publish_odom>true</publish_odom>
       <publish_odom_tf>true</publish_odom_tf>
-      <!-- odometry_topic>odom</odometry_topic -->
+      <odometry_topic>odom</odometry_topic>
       <!-- remapping>/odom:=/odom</remapping -->
       <odometry_frame>odom</odometry_frame>
       <robot_base_frame>base_footprint</robot_base_frame>
+      <!--odometry_source>1</odometry_source -->
     </plugin>
   </gazebo>
