Commit message: Add prefix to XACRO bin file

File: amrj16_bin_description/urdf/amrj16_empty_bin.xacro (robot description, xacro)
@@ -1,69 +1,71 @@
 <?xml version="1.0"?>
-    <robot xmlns:xacro="http://www.ros.org/wiki/xacro" name="empty_bin">
-    <link name="base_footprint">
-    </link>
-    <link name="base_link">
-    </link>
-    <joint name="base_link_base_footprintjoint" type="fixed">
-    <origin rpy="0 0 0" xyz="0 0 0.103" />
-    <parent link="base_footprint" />
-    <child link="base_link" />
-  </joint>
-    <!-- chassis-->
-    <link name="chassis">
-    <visual>
-      <origin xyz="0 0 0" rpy="0 0 0"/>
-      <geometry>
-        <mesh filename="package://amrj16_bin_description/models/meshes/utimac_bin_v1.dae"/>
-      </geometry>
-    </visual>
-    <collision>
-      <origin xyz="0 0 0" rpy="0 0 0"/>
-      <geometry>
-        <mesh filename="package://amrj16_bin_description/models/meshes/utimac_bin_v1.dae"/>
-      </geometry>
-    </collision>
-    <inertial>
-        <mass value="34.2"/>
-        <origin rpy="0 0 0" xyz="0 0 0"/>
-        <inertia ixx="10.164712" ixy="0.021460923" ixz="-0.0060724714" iyy="3.4403550" iyz="1.7125796" izz="12.572506"/>
-    </inertial>
-  </link>
-  <joint name="base_link_joint" type="fixed">
-    <origin rpy="0 0 0" xyz="0 0 0" />
-    <parent link="base_link" />
-    <child link="chassis" />
-  </joint>
+<robot xmlns:xacro="http://www.ros.org/wiki/xacro" name="empty_bin">
+    <!-- Definizione della variabile prefix -->
+    <xacro:property name="prefix" value="empty_bin"/>
+    <!-- Link e giunti con prefix -->
+    <link name="${prefix}_base_footprint">
+    </link>
+    <link name="${prefix}_base_link">
+    </link>
+    <joint name="${prefix}_base_link_base_footprintjoint" type="fixed">
+        <origin rpy="0 0 0" xyz="0 0 0.103" />
+        <parent link="${prefix}_base_footprint" />
+        <child link="${prefix}_base_link" />
+    </joint>
+    <!-- chassis -->
+    <link name="${prefix}_chassis">
+        <visual>
+            <origin xyz="0 0 0" rpy="0 0 0"/>
+            <geometry>
+                <mesh filename="package://amrj16_bin_description/models/meshes/utimac_bin_v1.dae"/>
+            </geometry>
+        </visual>
+        <collision>
+            <origin xyz="0 0 0" rpy="0 0 0"/>
+            <geometry>
+                <mesh filename="package://amrj16_bin_description/models/meshes/utimac_bin_v1.dae"/>
+            </geometry>
+        </collision>
+        <inertial>
+            <mass value="38"/>
+            <origin rpy="0 0 0" xyz="0 0 0"/>
+            <inertia ixx="8.1" ixy="0.00213" ixz="4.56" iyy="11.5" iyz="-0.00156" izz="7.71"/>
+        </inertial>
+    </link>
+    <joint name="${prefix}_base_link_joint" type="fixed">
+        <origin rpy="0 0 0" xyz="0 0 0" />
+        <parent link="${prefix}_base_link" />
+        <child link="${prefix}_chassis" />
+    </joint>
     <!-- front-right caster hub -->
-    <link name="front_right_caster_hub">
-        <visual>
-            <origin xyz="0 0 0" rpy="0 0 0"/>
-                <geometry>
-                    <mesh filename="package://amrj16_bin_description/models/meshes/utimac_caster_bin_v1.dae"/>
-                </geometry>
-        </visual>
-    <collision>
-        <origin xyz="0 0 0" rpy="0 0 0"/>
-        <geometry>
-                 <mesh filename="package://amrj16_bin_description/models/meshes/utimac_caster_bin_v1.dae"/>
-        </geometry>
-    </collision>
-    <inertial>
-        <mass value="1"/>
-        <origin rpy="0 0 0" xyz="0 0 0"/>
-        <inertia
-            ixx="0.00006" ixy="0.000000359" ixz="0.000014875" iyy="0.000059805" iyz="-0.00000077564" izz="0.000042536"/>
-    </inertial>
-    </link>
-    <joint name="chassis_front_right_caster_hub_joint" type="continuous">
+    <link name="${prefix}_front_right_caster_hub">
+        <visual>
+            <origin xyz="0 0 0" rpy="0 0 0"/>
+            <geometry>
+                <mesh filename="package://amrj16_bin_description/models/meshes/utimac_caster_bin_v1.dae"/>
+            </geometry>
+        </visual>
+        <collision>
+            <origin xyz="0 0 0" rpy="0 0 0"/>
+            <geometry>
+                <mesh filename="package://amrj16_bin_description/models/meshes/utimac_caster_bin_v1.dae"/>
+            </geometry>
+        </collision>
+        <inertial>
+            <mass value="0.5"/>
+            <origin rpy="0 0 0" xyz="0 0 0"/>
+            <inertia ixx="0.0008063" ixy="0.00000393" ixz="-0.00000650" iyy="0.000693" iyz="0.000265" izz="0.0005498"/>
+        </inertial>
+    </link>
+    <joint name="${prefix}_chassis_front_right_caster_hub_joint" type="continuous">
        <origin xyz="0.2925 0.215 0" rpy="0 0 0"/>
-        <parent link="chassis"/>
-        <child link="front_right_caster_hub"/>
+        <parent link="${prefix}_chassis"/>
+        <child link="${prefix}_front_right_caster_hub"/>
         <axis xyz="0 0 1"/>
         <limit effort="1000.0" velocity="100.0" />
-        <dynamics damping="0.0" friction="0.1"/>
-    </joint>
-    <!-- front-right caster wheel -->
-    <link name="front_right_caster_wheel">
+        <dynamics damping="0.5" friction="0.5"/>
+    </joint>
+ <!-- front-right caster wheel -->
+            <link name="${prefix}_front_right_caster_wheel">
         <visual>
             <origin xyz="0 0 0" rpy="1.57 0 0"/>
@@ -75,15 +77,15 @@
         <origin xyz="0 0 0" rpy="1.57  0 0"/>
         <geometry>
-                 <mesh filename="package://amrj16_bin_description/models/meshes/utimac_wheel_bin_v1.dae"/>
+                <cylinder radius="0.04" length="0.02"/>
         </geometry>
     </collision>
     <inertial>
-        <mass value="0.189"/>
+        <mass value="0.5"/>
         <origin rpy="0 0 0" xyz="1.57  0 0"/>
         <inertia
-            ixx="0.000025441" ixy="0" ixz="0" iyy="0.00002543" iyz="-0.0000000017817" izz="0.000028616"/>
+            ixx="0.0003265" ixy="0" ixz="0" iyy="0.0003265" iyz="0" izz="0.0005849"/>
     </inertial>
     </link>
-    <gazebo reference="front_right_caster_wheel">
+    <gazebo reference="${prefix}_front_right_caster_wheel">
         <kp>1000000000000000000000000000.0</kp>
         <kd>1000000000000000000000000000.0</kd>
@@ -91,43 +93,42 @@
         <mu2>10.0</mu2>
     </gazebo>
-    <joint name="front_right_caster_hub_wheel_joint" type="continuous">
+    <joint name="${prefix}_front_right_caster_hub_wheel_joint" type="continuous">
        <origin xyz="0.039 0 -0.067" rpy="0 0 0"/>
-        <parent link="front_right_caster_hub"/>
-        <child link="front_right_caster_wheel"/>
+        <parent link="${prefix}_front_right_caster_hub"/>
+        <child link="${prefix}_front_right_caster_wheel"/>
         <axis xyz="0 1 0"/>
         <limit effort="1000.0" velocity="100.0" />
-        <dynamics damping="0.0" friction="0.1"/>
-    </joint>
-    <!-- front-left caster hub -->
-    <link name="front_left_caster_hub">
-        <visual>
-            <origin xyz="0 0 0" rpy="0 0 0"/>
-                <geometry>
-                    <mesh filename="package://amrj16_bin_description/models/meshes/utimac_caster_bin_v1.dae"/>
-                </geometry>
-        </visual>
-        <collision>
-            <origin xyz="0 0 0" rpy="0 0 0"/>
-            <geometry>
-                    <mesh filename="package://amrj16_bin_description/models/meshes/utimac_caster_bin_v1.dae"/>
-            </geometry>
-        </collision>
-        <inertial>
-            <mass value="0.140"/>
-            <origin rpy="0 0 0" xyz="0 0 0"/>
-            <inertia
-                ixx="0.00006" ixy="0.000000359" ixz="0.000014875" iyy="0.000059805" iyz="-0.00000077564" izz="0.000042536"/>
-        </inertial>
-    </link>
-    <joint name="chassis_front_left_caster_hub_joint" type="continuous">
-        <origin xyz="0.2925 -0.215 0" rpy="0 0 0"/>
-        <parent link="chassis"/>
-        <child link="front_left_caster_hub"/>
+        <dynamics damping="0.5" friction="0.5"/>
+    </joint>
+ <!-- front-left caster hub -->
+    <link name="${prefix}_front_left_caster_hub">
+        <visual>
+            <origin xyz="0 0 0" rpy="0 0 0"/>
+            <geometry>
+                <mesh filename="package://amrj16_bin_description/models/meshes/utimac_caster_bin_v1.dae"/>
+            </geometry>
+        </visual>
+        <collision>
+            <origin xyz="0 0 0" rpy="0 0 0"/>
+            <geometry>
+                <mesh filename="package://amrj16_bin_description/models/meshes/utimac_caster_bin_v1.dae"/>
+            </geometry>
+        </collision>
+        <inertial>
+            <mass value="0.5"/>
+            <origin rpy="0 0 0" xyz="0 0 0"/>
+            <inertia ixx="0.0008063" ixy="0.00000393" ixz="-0.00000650" iyy="0.000693" iyz="0.000265" izz="0.0005498"/>
+        </inertial>
+    </link>
+    <joint name="${prefix}_chassis_front_left_caster_hub_joint" type="continuous">
+       <origin xyz="0.2925 -0.215 0" rpy="0 0 0"/>
+        <parent link="${prefix}_chassis"/>
+        <child link="${prefix}_front_left_caster_hub"/>
         <axis xyz="0 0 1"/>
         <limit effort="1000.0" velocity="100.0" />
-        <dynamics damping="0.0" friction="0.1"/>
-    </joint>
-    <!-- front-left caster wheel -->
-    <link name="front_left_caster_wheel">
+        <dynamics damping="0.5" friction="0.5"/>
+    </joint>
+<!-- front-left caster wheel -->
+            <link name="${prefix}_front_left_caster_wheel">
         <visual>
             <origin xyz="0 0 0" rpy="1.57 0 0"/>
@@ -136,18 +137,18 @@
                 </geometry>
         </visual>
-        <collision>
-            <origin xyz="0 0 0" rpy="1.57 0 0"/>
-            <geometry>
-                   <mesh filename="package://amrj16_bin_description/models/meshes/utimac_wheel_bin_v1.dae"/>
-            </geometry>
-        </collision>
-        <inertial>
-            <mass value="1"/>
-            <origin rpy="0 0 0" xyz="1.57 0 0"/>
-            <inertia
-                ixx="0.000025441" ixy="0" ixz="0" iyy="0.00002543" iyz="-0.0000000017817" izz="0.000028616"/>
-        </inertial>
-    </link>
-    <gazebo reference="front_left_caster_wheel">
+    <collision>
+        <origin xyz="0 0 0" rpy="1.57  0 0"/>
+        <geometry>
+                <cylinder radius="0.04" length="0.02"/>
+        </geometry>
+    </collision>
+    <inertial>
+        <mass value="0.5"/>
+        <origin rpy="0 0 0" xyz="1.57  0 0"/>
+        <inertia
+            ixx="0.0003265" ixy="0" ixz="0" iyy="0.0003265" iyz="0" izz="0.0005849"/>
+    </inertial>
+    </link>
+    <gazebo reference="${prefix}_front_left_caster_wheel">
         <kp>1000000000000000000000000000.0</kp>
         <kd>1000000000000000000000000000.0</kd>
@@ -155,43 +156,42 @@
         <mu2>10.0</mu2>
     </gazebo>
-    <joint name="front_left_caster_hub_wheel_joint" type="continuous">
-        <origin xyz="0.039 0 -0.067" rpy="0 0 0"/>
-        <parent link="front_left_caster_hub"/>
-        <child link="front_left_caster_wheel"/>
+    <joint name="${prefix}_front_left_caster_hub_wheel_joint" type="continuous">
+       <origin xyz="0.039 0 -0.067" rpy="0 0 0"/>
+        <parent link="${prefix}_front_left_caster_hub"/>
+        <child link="${prefix}_front_left_caster_wheel"/>
         <axis xyz="0 1 0"/>
         <limit effort="1000.0" velocity="100.0" />
-        <dynamics damping="0.0" friction="0.1"/>
-    </joint>
-    <!-- rear-right caster hub -->
-    <link name="rear_right_caster_hub">
-        <visual>
-            <origin xyz="0 0 0" rpy="0 0 0"/>
-                <geometry>
-                    <mesh filename="package://amrj16_bin_description/models/meshes/utimac_caster_bin_v1.dae"/>
-                </geometry>
-        </visual>
-    <collision>
-        <origin xyz="0 0 0" rpy="0 0 0"/>
-        <geometry>
-                 <mesh filename="package://amrj16_bin_description/models/meshes/utimac_caster_bin_v1.dae"/>
-        </geometry>
-    </collision>
-    <inertial>
-        <mass value="1"/>
-        <origin rpy="0 0 0" xyz="0 0 0"/>
-        <inertia
-            ixx="0.00006" ixy="0.000000359" ixz="0.000014875" iyy="0.000059805" iyz="-0.00000077564" izz="0.000042536"/>
-    </inertial>
-    </link>
-    <joint name="chassis_rear_right_caster_hub_joint" type="continuous">
+        <dynamics damping="0.5" friction="0.5"/>
+    </joint>
+  <!-- rear-right caster hub -->
+    <link name="${prefix}_rear_right_caster_hub">
+        <visual>
+            <origin xyz="0 0 0" rpy="0 0 0"/>
+            <geometry>
+                <mesh filename="package://amrj16_bin_description/models/meshes/utimac_caster_bin_v1.dae"/>
+            </geometry>
+        </visual>
+        <collision>
+            <origin xyz="0 0 0" rpy="0 0 0"/>
+            <geometry>
+                <mesh filename="package://amrj16_bin_description/models/meshes/utimac_caster_bin_v1.dae"/>
+            </geometry>
+        </collision>
+        <inertial>
+            <mass value="0.5"/>
+            <origin rpy="0 0 0" xyz="0 0 0"/>
+            <inertia ixx="0.0008063" ixy="0.00000393" ixz="-0.00000650" iyy="0.000693" iyz="0.000265" izz="0.0005498"/>
+        </inertial>
+    </link>
+    <joint name="${prefix}_chassis_rear_right_caster_hub_joint" type="continuous">
        <origin xyz="-0.2925 0.215 0" rpy="0 0 0"/>
-        <parent link="chassis"/>
-        <child link="rear_right_caster_hub"/>
+        <parent link="${prefix}_chassis"/>
+        <child link="${prefix}_rear_right_caster_hub"/>
         <axis xyz="0 0 1"/>
         <limit effort="1000.0" velocity="100.0" />
-        <dynamics damping="0.0" friction="0.1"/>
+        <dynamics damping="0.5" friction="0.5"/>
     </joint>
  <!-- rear-right caster wheel -->
-    <link name="rear_right_caster_wheel">
+            <link name="${prefix}_rear_right_caster_wheel">
         <visual>
             <origin xyz="0 0 0" rpy="1.57 0 0"/>
@@ -203,15 +203,15 @@
         <origin xyz="0 0 0" rpy="1.57  0 0"/>
         <geometry>
-                 <mesh filename="package://amrj16_bin_description/models/meshes/utimac_wheel_bin_v1.dae"/>
+                <cylinder radius="0.04" length="0.02"/>
         </geometry>
     </collision>
     <inertial>
-        <mass value="1"/>
+        <mass value="0.5"/>
         <origin rpy="0 0 0" xyz="1.57  0 0"/>
         <inertia
-            ixx="0.000025441" ixy="0" ixz="0" iyy="0.00002543" iyz="-0.0000000017817" izz="0.000028616"/>
+            ixx="0.0003265" ixy="0" ixz="0" iyy="0.0003265" iyz="0" izz="0.0005849"/>
     </inertial>
     </link>
-    <gazebo reference="rear_right_caster_wheel">
+   <gazebo reference="${prefix}_rear_right_caster_wheel">
         <kp>1000000000000000000000000000.0</kp>
         <kd>1000000000000000000000000000.0</kd>
@@ -219,44 +219,42 @@
         <mu2>10.0</mu2>
     </gazebo>
-    <joint name="rear_right_caster_hub_wheel_joint" type="continuous">
+    <joint name="${prefix}_rear_right_caster_hub_wheel_joint" type="continuous">
        <origin xyz="0.039 0 -0.067" rpy="0 0 0"/>
-        <parent link="rear_right_caster_hub"/>
-        <child link="rear_right_caster_wheel"/>
+        <parent link="${prefix}_rear_right_caster_hub"/>
+        <child link="${prefix}_rear_right_caster_wheel"/>
         <axis xyz="0 1 0"/>
         <limit effort="1000.0" velocity="100.0" />
-        <dynamics damping="0.0" friction="0.1"/>
-    </joint>
-=======================
- <!-- rear-left caster hub -->
-    <link name="rear_left_caster_hub">
-        <visual>
-            <origin xyz="0 0 0" rpy="0 0 0"/>
-                <geometry>
-                    <mesh filename="package://amrj16_bin_description/models/meshes/utimac_caster_bin_v1.dae"/>
-                </geometry>
-        </visual>
-    <collision>
-        <origin xyz="0 0 0" rpy="0 0 0"/>
-        <geometry>
-                 <mesh filename="package://amrj16_bin_description/models/meshes/utimac_caster_bin_v1.dae"/>
-        </geometry>
-    </collision>
-    <inertial>
-        <mass value="1"/>
-        <origin rpy="0 0 0" xyz="0 0 0"/>
-        <inertia
-            ixx="0.00006" ixy="0.000000359" ixz="0.000014875" iyy="0.000059805" iyz="-0.00000077564" izz="0.000042536"/>
-    </inertial>
-    </link>
-    <joint name="chassis_rear_left_caster_hub_joint" type="continuous">
+        <dynamics damping="0.5" friction="0.5"/>
+    </joint>
+<!-- rear-left caster hub -->
+    <link name="${prefix}_rear_left_caster_hub">
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