Commit message: Rewrite full and empty bin xacro code

File: amrj16_bin_description/urdf/amrj16_empty_bin.xacro (robot description, xacro)
@@ -3,5 +3,4 @@
     <!-- Definizione della variabile prefix -->
     <xacro:property name="prefix" value="empty_bin"/>
-    <!-- Link e giunti con prefix -->
     <link name="${prefix}_base_footprint">
     </link>
@@ -13,24 +12,24 @@
         <child link="${prefix}_base_link" />
     </joint>
-    <!-- chassis -->
+    <!-- chassis-->
     <link name="${prefix}_chassis">
-        <visual>
-            <origin xyz="0 0 0" rpy="0 0 0"/>
-            <geometry>
-                <mesh filename="package://amrj16_bin_description/models/meshes/utimac_bin_v1.dae"/>
-            </geometry>
-        </visual>
-        <collision>
-            <origin xyz="0 0 0" rpy="0 0 0"/>
-            <geometry>
-                <mesh filename="package://amrj16_bin_description/models/meshes/utimac_bin_v1.dae"/>
-            </geometry>
-        </collision>
-        <inertial>
-            <mass value="38"/>
-            <origin rpy="0 0 0" xyz="0 0 0"/>
-            <inertia ixx="8.1" ixy="0.00213" ixz="4.56" iyy="11.5" iyz="-0.00156" izz="7.71"/>
-        </inertial>
-    </link>
+    <visual>
+      <origin xyz="0 0 0" rpy="0 0 0"/>
+      <geometry>
+        <mesh filename="package://amrj16_bin_description/models/meshes/utimac_bin_v1.dae"/>
+      </geometry>
+    </visual>
+    <collision>
+      <origin xyz="0 0 0" rpy="0 0 0"/>
+      <geometry>
+       <mesh filename="package://amrj16_bin_description/models/meshes/utimac_bin_v1.dae"/>
+      </geometry>
+    </collision>
+    <inertial>
+        <mass value="38"/>
+        <origin rpy="0 0 0" xyz="-0.1055 0 -0.0199"/>
+        <inertia ixx="8.1" ixy="0.00213" ixz="4.56" iyy="11.5" iyz="-0.00156" izz="7.71"/>
+    </inertial>
+  </link>
     <joint name="${prefix}_base_link_joint" type="fixed">
         <origin rpy="0 0 0" xyz="0 0 0" />
@@ -42,7 +41,69 @@
         <visual>
             <origin xyz="0 0 0" rpy="0 0 0"/>
-            <geometry>
+                <geometry>
+                    <mesh filename="package://amrj16_bin_description/models/meshes/utimac_caster_bin_v1.dae"/>
+                </geometry>
+        </visual>
+    <collision>
+        <origin xyz="0 0 0" rpy="0 0 0"/>
+        <geometry>
                 <mesh filename="package://amrj16_bin_description/models/meshes/utimac_caster_bin_v1.dae"/>
-            </geometry>
+        </geometry>
+    </collision>
+    <inertial>
+        <mass value="0.7"/>
+        <origin rpy="0 0 0" xyz="0 0 0"/>
+        <inertia
+            ixx="0.0008063" ixy="0.00000393" ixz="-0.00000650" iyy="0.000693" iyz="0.000265" izz="0.0005498"/>
+    </inertial>
+    </link>
+    <joint name="${prefix}_chassis_front_right_caster_hub_joint" type="continuous">
+        <origin xyz="0.2925 0.215 0" rpy="0 0 0"/>
+        <parent link="${prefix}_chassis"/>
+        <child link="${prefix}_front_right_caster_hub"/>
+        <axis xyz="0 0 1"/>
+        <dynamics damping="0.5" friction="0.5"/>
+    </joint>
+    <!-- front-right caster wheel -->
+    <link name="${prefix}_front_right_caster_wheel">
+        <visual>
+            <origin xyz="0 0 0" rpy="0 0 0"/>
+                <geometry>
+                    <mesh filename="package://amrj16_bin_description/models/meshes/utimac_wheel_bin_v1.dae"/>
+                </geometry>
+        </visual>
+    <collision>
+        <origin xyz="0 0 0" rpy="0 0 0"/>
+        <geometry>
+            <cylinder radius="0.040" length="0.02"/>
+        </geometry>
+    </collision>
+    <inertial>
+        <mass value="0.5"/>
+        <origin  xyz="0 0 0" rpy="0 0 0"/>
+        <inertia
+           ixx="0.0003265" ixy="0" ixz="0" iyy="0.0003265" iyz="0" izz="0.0005849"/>
+    </inertial>
+    </link>
+    <gazebo reference="${prefix}_front_right_caster_wheel">
+        <kp>5000000000</kp>
+        <kd>5000000000</kd>
+        <mu1>10.0</mu1>
+        <mu2>10.0</mu2>
+    </gazebo>
+    <joint name="${prefix}_front_right_caster_hub_wheel_joint" type="continuous">
+        <origin xyz="0.039 0 -0.067" rpy="1.57 0 0"/>
+        <parent link="${prefix}_front_right_caster_hub"/>
+        <child link="${prefix}_front_right_caster_wheel"/>
+        <axis xyz="0 0 1"/>
+        <dynamics damping="0.5" friction="0.5"/>
+    </joint>
+    <!-- front-left caster hub -->
+    <link name="${prefix}_front_left_caster_hub">
+        <visual>
+            <origin xyz="0 0 0" rpy="0 0 0"/>
+                <geometry>
+                    <mesh filename="package://amrj16_bin_description/models/meshes/utimac_caster_bin_v1.dae"/>
+                </geometry>
         </visual>
         <collision>
@@ -55,60 +116,27 @@
             <mass value="0.7"/>
             <origin rpy="0 0 0" xyz="0 0 0"/>
-            <inertia ixx="0.0008063" ixy="0.00000393" ixz="-0.00000650" iyy="0.000693" iyz="0.000265" izz="0.0005498"/>
+            <inertia
+                 ixx="0.0008063" ixy="0.00000393" ixz="-0.00000650" iyy="0.000693" iyz="0.000265" izz="0.0005498"/>
         </inertial>
     </link>
-    <joint name="${prefix}_chassis_front_right_caster_hub_joint" type="continuous">
-       <origin xyz="0.2925 0.215 0" rpy="0 0 0"/>
+    <joint name="${prefix}_chassis_front_left_caster_hub_joint" type="continuous">
+        <origin xyz="0.2925 -0.215 0" rpy="0 0 0"/>
         <parent link="${prefix}_chassis"/>
-        <child link="${prefix}_front_right_caster_hub"/>
-        <axis xyz="0 0 1"/>
-        <dynamics damping="0.5" friction="0.1"/>
-    </joint>
- <!-- front-right caster wheel -->
-            <link name="${prefix}_front_right_caster_wheel">
-        <visual>
-            <origin xyz="0 0 0" rpy="1.57 0 0"/>
+        <child link="${prefix}_front_left_caster_hub"/>
+        <axis xyz="0 0 1"/>
+        <dynamics damping="0.5" friction="0.5"/>
+    </joint>
+    <!-- front-left caster wheel -->
+    <link name="${prefix}_front_left_caster_wheel">
+        <visual>
+            <origin xyz="0 0 0" rpy="0 0 0"/>
                 <geometry>
                     <mesh filename="package://amrj16_bin_description/models/meshes/utimac_wheel_bin_v1.dae"/>
                 </geometry>
         </visual>
-    <collision>
-        <origin xyz="0 0 0" rpy="1.57  0 0"/>
-        <geometry>
-                <cylinder radius="0.04" length="0.02"/>
-        </geometry>
-    </collision>
-    <inertial>
-        <mass value="0.7"/>
-        <origin rpy="0 0 0" xyz="1.57  0 0"/>
-        <inertia
-            ixx="0.0003265" ixy="0" ixz="0" iyy="0.0003265" iyz="0" izz="0.0005849"/>
-    </inertial>
-    </link>
-    <gazebo reference="${prefix}_front_right_caster_wheel">
-        <kp>1000000000000000000000000000.0</kp>
-        <kd>1000000000000000000000000000.0</kd>
-        <mu1>10.0</mu1>
-        <mu2>10.0</mu2>
-    </gazebo>
-    <joint name="${prefix}_front_right_caster_hub_wheel_joint" type="continuous">
-       <origin xyz="0.039 0 -0.067" rpy="0 0 0"/>
-        <parent link="${prefix}_front_right_caster_hub"/>
-        <child link="${prefix}_front_right_caster_wheel"/>
-        <axis xyz="0 1 0"/>
-        <dynamics damping="0.5" friction="0.1"/>
-    </joint>
- <!-- front-left caster hub -->
-    <link name="${prefix}_front_left_caster_hub">
-        <visual>
+        <collision>
             <origin xyz="0 0 0" rpy="0 0 0"/>
             <geometry>
-                <mesh filename="package://amrj16_bin_description/models/meshes/utimac_caster_bin_v1.dae"/>
-            </geometry>
-        </visual>
-        <collision>
-            <origin xyz="0 0 0" rpy="0 0 0"/>
-            <geometry>
-                <mesh filename="package://amrj16_bin_description/models/meshes/utimac_caster_bin_v1.dae"/>
+                <cylinder radius="0.040" length="0.02"/>
             </geometry>
         </collision>
@@ -116,56 +144,90 @@
             <mass value="0.5"/>
             <origin rpy="0 0 0" xyz="0 0 0"/>
-            <inertia ixx="0.0008063" ixy="0.00000393" ixz="-0.00000650" iyy="0.000693" iyz="0.000265" izz="0.0005498"/>
+            <inertia
+                ixx="0.0003265" ixy="0" ixz="0" iyy="0.0003265" iyz="0" izz="0.0005849"/>
         </inertial>
     </link>
-    <joint name="${prefix}_chassis_front_left_caster_hub_joint" type="continuous">
-       <origin xyz="0.2925 -0.215 0" rpy="0 0 0"/>
-        <parent link="${prefix}_chassis"/>
-        <child link="${prefix}_front_left_caster_hub"/>
-        <axis xyz="0 0 1"/>
-        <limit effort="1000.0" velocity="100.0" />
-        <dynamics damping="0.5" friction="0.1"/>
-    </joint>
-<!-- front-left caster wheel -->
-            <link name="${prefix}_front_left_caster_wheel">
-        <visual>
-            <origin xyz="0 0 0" rpy="1.57 0 0"/>
-                <geometry>
-                    <mesh filename="package://amrj16_bin_description/models/meshes/utimac_wheel_bin_v1.dae"/>
-                </geometry>
-        </visual>
-    <collision>
-        <origin xyz="0 0 0" rpy="1.57  0 0"/>
-        <geometry>
-                <cylinder radius="0.04" length="0.02"/>
-        </geometry>
-    </collision>
-    <inertial>
-        <mass value="0.7"/>
-        <origin rpy="0 0 0" xyz="1.57  0 0"/>
-        <inertia
-            ixx="0.0003265" ixy="0" ixz="0" iyy="0.0003265" iyz="0" izz="0.0005849"/>
-    </inertial>
-    </link>
     <gazebo reference="${prefix}_front_left_caster_wheel">
-        <kp>1000000000000000000000000000.0</kp>
-        <kd>1000000000000000000000000000.0</kd>
+        <kp>5000000000</kp>
+        <kd>5000000000</kd>
         <mu1>10.0</mu1>
         <mu2>10.0</mu2>
     </gazebo>
     <joint name="${prefix}_front_left_caster_hub_wheel_joint" type="continuous">
-       <origin xyz="0.039 0 -0.067" rpy="0 0 0"/>
+       <origin xyz="0.039 0 -0.067" rpy="1.57 0 0"/>
         <parent link="${prefix}_front_left_caster_hub"/>
         <child link="${prefix}_front_left_caster_wheel"/>
-        <axis xyz="0 1 0"/>
-        <dynamics damping="0.5" friction="0.1"/>
-    </joint>
-  <!-- rear-right caster hub -->
+        <axis xyz="0 0 1"/>
+        <dynamics damping="0.5" friction="0.5"/>
+    </joint>
+ <!-- rear-right caster hub -->
     <link name="${prefix}_rear_right_caster_hub">
         <visual>
             <origin xyz="0 0 0" rpy="0 0 0"/>
-            <geometry>
+                <geometry>
+                    <mesh filename="package://amrj16_bin_description/models/meshes/utimac_caster_bin_v1.dae"/>
+                </geometry>
+        </visual>
+    <collision>
+        <origin xyz="0 0 0" rpy="0 0 0"/>
+        <geometry>
                 <mesh filename="package://amrj16_bin_description/models/meshes/utimac_caster_bin_v1.dae"/>
-            </geometry>
+        </geometry>
+    </collision>
+    <inertial>
+        <mass value="0.7"/>
+        <origin rpy="0 0 0" xyz="0 0 0"/>
+        <inertia
+           ixx="0.0008063" ixy="0.00000393" ixz="-0.00000650" iyy="0.000693" iyz="0.000265" izz="0.0005498"/>
+    </inertial>
+    </link>
+    <joint name="${prefix}_chassis_rear_right_caster_hub_joint" type="continuous">
+       <origin xyz="-0.2925 0.215 0" rpy="0 0 0"/>
+        <parent link="${prefix}_chassis"/>
+        <child link="${prefix}_rear_right_caster_hub"/>
+        <axis xyz="0 0 1"/>
+        <dynamics damping="0.5" friction="0.5"/>
+    </joint>
+    <!-- rear-right caster wheel -->
+    <link name="${prefix}_rear_right_caster_wheel">
+        <visual>
+            <origin xyz="0 0 0" rpy="0 0 0"/>
+                <geometry>
+                    <mesh filename="package://amrj16_bin_description/models/meshes/utimac_wheel_bin_v1.dae"/>
+                </geometry>
+        </visual>
+    <collision>
+        <origin xyz="0 0 0" rpy="0 0 0"/>
+        <geometry>
+            <cylinder radius="0.040" length="0.02"/>
+        </geometry>
+    </collision>
+    <inertial>
+        <mass value="0.5"/>
+        <origin rpy="0 0 0" xyz="0 0 0"/>
+        <inertia
+           ixx="0.0003265" ixy="0" ixz="0" iyy="0.0003265" iyz="0" izz="0.0005849"/>
+    </inertial>
+    </link>
+    <gazebo reference="${prefix}_rear_right_caster_wheel">
+        <kp>5000000000</kp>
+        <kd>5000000000</kd>
+        <mu1>10.0</mu1>
+        <mu2>10.0</mu2>
+    </gazebo>
+    <joint name="${prefix}_rear_right_caster_hub_wheel_joint" type="continuous">
+       <origin xyz="0.039 0 -0.067" rpy="1.57 0 0"/>
+        <parent link="${prefix}_rear_right_caster_hub"/>
+        <child link="${prefix}_rear_right_caster_wheel"/>
+        <axis xyz="0 0 1"/>
+        <dynamics damping="0.5" friction="0.5"/>
+    </joint>
+ <!-- rear-left caster hub -->
+    <link name="${prefix}_rear_left_caster_hub">
+        <visual>
+            <origin xyz="0 0 0" rpy="0 0 0"/>
+                <geometry>
+                    <mesh filename="package://amrj16_bin_description/models/meshes/utimac_caster_bin_v1.dae"/>
+                </geometry>
         </visual>
         <collision>
@@ -178,60 +240,27 @@
             <mass value="0.7"/>
             <origin rpy="0 0 0" xyz="0 0 0"/>
-            <inertia ixx="0.0008063" ixy="0.00000393" ixz="-0.00000650" iyy="0.000693" iyz="0.000265" izz="0.0005498"/>
+            <inertia
+                ixx="0.0008063" ixy="0.00000393" ixz="-0.00000650" iyy="0.000693" iyz="0.000265" izz="0.0005498"/>
         </inertial>
     </link>
-    <joint name="${prefix}_chassis_rear_right_caster_hub_joint" type="continuous">
-       <origin xyz="-0.2925 0.215 0" rpy="0 0 0"/>
+    <joint name="${prefix}_chassis_rear_left_caster_hub_joint" type="continuous">
+       <origin xyz="-0.2925 -0.215 0" rpy="0 0 0"/>
         <parent link="${prefix}_chassis"/>
-        <child link="${prefix}_rear_right_caster_hub"/>
-        <axis xyz="0 0 1"/>
-        <dynamics damping="0.5" friction="0.1"/>
-    </joint>
- <!-- rear-right caster wheel -->
-            <link name="${prefix}_rear_right_caster_wheel">
-        <visual>
-            <origin xyz="0 0 0" rpy="1.57 0 0"/>
+        <child link="${prefix}_rear_left_caster_hub"/>
+        <axis xyz="0 0 1"/>
+        <dynamics damping="0.5" friction="0.5"/>
+    </joint>
+    <!-- rear-left caster wheel -->
+    <link name="${prefix}_rear_left_caster_wheel">
+        <visual>
+            <origin xyz="0 0 0" rpy="0 0 0"/>
                 <geometry>
                     <mesh filename="package://amrj16_bin_description/models/meshes/utimac_wheel_bin_v1.dae"/>
                 </geometry>
         </visual>
-    <collision>
-        <origin xyz="0 0 0" rpy="1.57  0 0"/>
-        <geometry>
-                <cylinder radius="0.04" length="0.02"/>
-        </geometry>
-    </collision>
-    <inertial>
-        <mass value="0.5"/>
-        <origin rpy="0 0 0" xyz="1.57  0 0"/>
-        <inertia
-            ixx="0.0003265" ixy="0" ixz="0" iyy="0.0003265" iyz="0" izz="0.0005849"/>
-    </inertial>
-    </link>
-   <gazebo reference="${prefix}_rear_right_caster_wheel">
-        <kp>1000000000000000000000000000.0</kp>
-        <kd>1000000000000000000000000000.0</kd>
-        <mu1>10.0</mu1>
-        <mu2>10.0</mu2>
-    </gazebo>
-    <joint name="${prefix}_rear_right_caster_hub_wheel_joint" type="continuous">
-       <origin xyz="0.039 0 -0.067" rpy="0 0 0"/>
-        <parent link="${prefix}_rear_right_caster_hub"/>
-        <child link="${prefix}_rear_right_caster_wheel"/>
-        <axis xyz="0 1 0"/>
-        <dynamics damping="0.5" friction="0.1"/>
-    </joint>
-<!-- rear-left caster hub -->
-    <link name="${prefix}_rear_left_caster_hub">
-        <visual>
+        <collision>
             <origin xyz="0 0 0" rpy="0 0 0"/>
             <geometry>
-                <mesh filename="package://amrj16_bin_description/models/meshes/utimac_caster_bin_v1.dae"/>
-            </geometry>
-        </visual>
-        <collision>
-            <origin xyz="0 0 0" rpy="0 0 0"/>
-            <geometry>
-                <mesh filename="package://amrj16_bin_description/models/meshes/utimac_caster_bin_v1.dae"/>
+                <cylinder radius="0.040" length="0.02"/>
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