Commit message: Rewrite full and empty bin xacro code

File: amrj16_bin_description/urdf/amrj16_full_bin.xacro (robot description, xacro)
@@ -3,5 +3,4 @@
     <!-- Definizione della variabile prefix -->
     <xacro:property name="prefix" value="full_bin"/>
-    <!-- Link e giunti con prefix -->
     <link name="${prefix}_base_footprint">
     </link>
@@ -13,24 +12,24 @@
         <child link="${prefix}_base_link" />
     </joint>
-    <!-- chassis -->
+    <!-- chassis-->
     <link name="${prefix}_chassis">
-        <visual>
-            <origin xyz="0 0 0" rpy="0 0 0"/>
-            <geometry>
-                <mesh filename="package://amrj16_bin_description/models/meshes/utimac_bin_v1.dae"/>
-            </geometry>
-        </visual>
-        <collision>
-            <origin xyz="0 0 0.2" rpy="0 0 0"/>
-            <geometry>
-                <box size="0.815 0.690 0.293" />
-            </geometry>
-        </collision>
-        <inertial>
-            <mass value="38"/>
-            <origin  xyz="0 0 0" rpy="0 0 0"/>
-            <inertia ixx="8.1" ixy="0.00213" ixz="4.56" iyy="11.5" iyz="-0.00156" izz="7.71"/>
-        </inertial>
-    </link>
+    <visual>
+      <origin xyz="0 0 0" rpy="0 0 0"/>
+      <geometry>
+        <mesh filename="package://amrj16_bin_description/models/meshes/utimac_bin_v1.dae"/>
+      </geometry>
+    </visual>
+    <collision>
+      <origin xyz="0 0 0" rpy="0 0 0"/>
+      <geometry>
+       <mesh filename="package://amrj16_bin_description/models/meshes/utimac_bin_v1.dae"/>
+      </geometry>
+    </collision>
+    <inertial>
+        <mass value="38"/>
+        <origin rpy="0 0 0" xyz="-0.1055 0 -0.0199"/>
+        <inertia ixx="8.1" ixy="0.00213" ixz="4.56" iyy="11.5" iyz="-0.00156" izz="7.71"/>
+    </inertial>
+  </link>
     <joint name="${prefix}_base_link_joint" type="fixed">
         <origin rpy="0 0 0" xyz="0 0 0" />
@@ -42,163 +41,144 @@
         <visual>
             <origin xyz="0 0 0" rpy="0 0 0"/>
+                <geometry>
+                    <mesh filename="package://amrj16_bin_description/models/meshes/utimac_caster_bin_v1.dae"/>
+                </geometry>
+        </visual>
+    <collision>
+        <origin xyz="0 0 0" rpy="0 0 0"/>
+        <geometry>
+                <mesh filename="package://amrj16_bin_description/models/meshes/utimac_caster_bin_v1.dae"/>
+        </geometry>
+    </collision>
+    <inertial>
+        <mass value="0.7"/>
+        <origin rpy="0 0 0" xyz="0 0 0"/>
+        <inertia
+            ixx="0.0008063" ixy="0.00000393" ixz="-0.00000650" iyy="0.000693" iyz="0.000265" izz="0.0005498"/>
+    </inertial>
+    </link>
+    <joint name="${prefix}_chassis_front_right_caster_hub_joint" type="continuous">
+        <origin xyz="0.2925 0.215 0" rpy="0 0 0"/>
+        <parent link="${prefix}_chassis"/>
+        <child link="${prefix}_front_right_caster_hub"/>
+        <axis xyz="0 0 1"/>
+        <dynamics damping="0.5" friction="0.5"/>
+    </joint>
+    <!-- front-right caster wheel -->
+    <link name="${prefix}_front_right_caster_wheel">
+        <visual>
+            <origin xyz="0 0 0" rpy="0 0 0"/>
+                <geometry>
+                    <mesh filename="package://amrj16_bin_description/models/meshes/utimac_wheel_bin_v1.dae"/>
+                </geometry>
+        </visual>
+    <collision>
+        <origin xyz="0 0 0" rpy="0 0 0"/>
+        <geometry>
+            <cylinder radius="0.040" length="0.02"/>
+        </geometry>
+    </collision>
+    <inertial>
+        <mass value="0.5"/>
+        <origin  xyz="0 0 0" rpy="0 0 0"/>
+        <inertia
+           ixx="0.0003265" ixy="0" ixz="0" iyy="0.0003265" iyz="0" izz="0.0005849"/>
+    </inertial>
+    </link>
+    <gazebo reference="${prefix}_front_right_caster_wheel">
+        <kp>5000000000</kp>
+        <kd>5000000000</kd>
+        <mu1>10.0</mu1>
+        <mu2>10.0</mu2>
+    </gazebo>
+    <joint name="${prefix}_front_right_caster_hub_wheel_joint" type="continuous">
+        <origin xyz="0.039 0 -0.067" rpy="1.57 0 0"/>
+        <parent link="${prefix}_front_right_caster_hub"/>
+        <child link="${prefix}_front_right_caster_wheel"/>
+        <axis xyz="0 0 1"/>
+        <dynamics damping="0.5" friction="0.5"/>
+    </joint>
+    <!-- front-left caster hub -->
+    <link name="${prefix}_front_left_caster_hub">
+        <visual>
+            <origin xyz="0 0 0" rpy="0 0 0"/>
+                <geometry>
+                    <mesh filename="package://amrj16_bin_description/models/meshes/utimac_caster_bin_v1.dae"/>
+                </geometry>
+        </visual>
+        <collision>
+            <origin xyz="0 0 0" rpy="0 0 0"/>
             <geometry>
                 <mesh filename="package://amrj16_bin_description/models/meshes/utimac_caster_bin_v1.dae"/>
             </geometry>
-        </visual>
-        <!--collision>
-            <origin xyz="0 0 0" rpy="0 0 0"/>
-            <geometry>
-                <mesh filename="package://amrj16_bin_description/models/meshes/utimac_caster_bin_v1.dae"/>
-            </geometry>
-        </collision -->
+        </collision>
         <inertial>
-            <mass value="1"/>
+            <mass value="0.7"/>
             <origin rpy="0 0 0" xyz="0 0 0"/>
-            <inertia ixx="0.0008063" ixy="0.00000393" ixz="-0.00000650" iyy="0.000693" iyz="0.000265" izz="0.0005498"/>
+            <inertia
+                 ixx="0.0008063" ixy="0.00000393" ixz="-0.00000650" iyy="0.000693" iyz="0.000265" izz="0.0005498"/>
         </inertial>
     </link>
-    <joint name="${prefix}_chassis_front_right_caster_hub_joint" type="continuous">
-       <origin xyz="0.2925 0.215 0" rpy="0 0 0"/>
-        <parent link="${prefix}_chassis"/>
-        <child link="${prefix}_front_right_caster_hub"/>
-        <axis xyz="0 0 1"/>
-              <dynamics damping="0.5" friction="0.1"/>
-    </joint>
- <!-- front-right caster wheel -->
-            <link name="${prefix}_front_right_caster_wheel">
-        <visual>
-            <origin xyz="0 0 0" rpy="1.57 0 0"/>
-                <geometry>
-                    <mesh filename="package://amrj16_bin_description/models/meshes/utimac_wheel_bin_v1.dae"/>
-                </geometry>
-        </visual>
-    <collision>
-        <origin xyz="0 0 0" rpy="1.57  0 0"/>
-        <geometry>
-                <cylinder radius="0.04" length="0.02"/>
-        </geometry>
-    </collision>
-    <inertial>
-        <mass value="1"/>
-        <origin rpy="0 0 0" xyz="1.57  0 0"/>
-        <inertia
-            ixx="0.0003265" ixy="0" ixz="0" iyy="0.0003265" iyz="0" izz="0.0005849"/>
-    </inertial>
-    </link>
-    <gazebo reference="${prefix}_front_right_caster_wheel">
-      <collision>
-        <surface>
-          <friction>
-            <ode>
-              <mu>0.3</mu>
-              <mu2>0.3</mu2>
-            </ode>
-            <bullet>
-              <friction>0.3</friction>
-              <friction2>0.3</friction2>
-              <rolling_friction>0.1</rolling_friction>
-            </bullet>
-          </friction>
-        </surface>
-      </collision>
-    </gazebo>
-    <joint name="${prefix}_front_right_caster_hub_wheel_joint" type="continuous">
-       <origin xyz="0.039 0 -0.067" rpy="0 0 0"/>
-        <parent link="${prefix}_front_right_caster_hub"/>
-        <child link="${prefix}_front_right_caster_wheel"/>
-        <axis xyz="0 1 0"/>
-        <dynamics damping="0.5" friction="1.5"/>
-    </joint>
- <!-- front-left caster hub -->
-    <link name="${prefix}_front_left_caster_hub">
-        <visual>
-            <origin xyz="0 0 0" rpy="0 0 0"/>
-            <geometry>
-                <mesh filename="package://amrj16_bin_description/models/meshes/utimac_caster_bin_v1.dae"/>
-            </geometry>
-        </visual>
-        <!--collision>
-            <origin xyz="0 0 0" rpy="0 0 0"/>
-            <geometry>
-                <mesh filename="package://amrj16_bin_description/models/meshes/utimac_caster_bin_v1.dae"/>
-            </geometry>
-        </collision -->
-        <inertial>
-            <mass value="1"/>
-            <origin rpy="0 0 0" xyz="0 0 0"/>
-            <inertia ixx="0.0008063" ixy="0.00000393" ixz="-0.00000650" iyy="0.000693" iyz="0.000265" izz="0.0005498"/>
-        </inertial>
-    </link>
     <joint name="${prefix}_chassis_front_left_caster_hub_joint" type="continuous">
-       <origin xyz="0.2925 -0.215 0" rpy="0 0 0"/>
+        <origin xyz="0.2925 -0.215 0" rpy="0 0 0"/>
         <parent link="${prefix}_chassis"/>
         <child link="${prefix}_front_left_caster_hub"/>
         <axis xyz="0 0 1"/>
-        <dynamics damping="0.5" friction="0.1"/>
-    </joint>
-<!-- front-left caster wheel -->
-            <link name="${prefix}_front_left_caster_wheel">
-        <visual>
-            <origin xyz="0 0 0" rpy="1.57 0 0"/>
+        <dynamics damping="0.5" friction="0.5"/>
+    </joint>
+    <!-- front-left caster wheel -->
+    <link name="${prefix}_front_left_caster_wheel">
+        <visual>
+            <origin xyz="0 0 0" rpy="0 0 0"/>
                 <geometry>
                     <mesh filename="package://amrj16_bin_description/models/meshes/utimac_wheel_bin_v1.dae"/>
                 </geometry>
         </visual>
-    <collision>
-        <origin xyz="0 0 0" rpy="1.57  0 0"/>
-        <geometry>
-                <cylinder radius="0.04" length="0.02"/>
-        </geometry>
-    </collision>
-    <inertial>
-        <mass value="1"/>
-        <origin rpy="0 0 0" xyz="1.57  0 0"/>
-        <inertia
-            ixx="0.0003265" ixy="0" ixz="0" iyy="0.0003265" iyz="0" izz="0.0005849"/>
-    </inertial>
+        <collision>
+            <origin xyz="0 0 0" rpy="0 0 0"/>
+            <geometry>
+                <cylinder radius="0.040" length="0.02"/>
+            </geometry>
+        </collision>
+        <inertial>
+            <mass value="0.5"/>
+            <origin rpy="0 0 0" xyz="0 0 0"/>
+            <inertia
+                ixx="0.0003265" ixy="0" ixz="0" iyy="0.0003265" iyz="0" izz="0.0005849"/>
+        </inertial>
     </link>
     <gazebo reference="${prefix}_front_left_caster_wheel">
-      <collision>
-        <surface>
-          <friction>
-            <ode>
-              <mu>0.3</mu>
-              <mu2>0.3</mu2>
-            </ode>
-            <bullet>
-              <friction>0.3</friction>
-              <friction2>0.3</friction2>
-              <rolling_friction>0.1</rolling_friction>
-            </bullet>
-          </friction>
-        </surface>
-      </collision>
+        <kp>5000000000</kp>
+        <kd>5000000000</kd>
+        <mu1>10.0</mu1>
+        <mu2>10.0</mu2>
     </gazebo>
     <joint name="${prefix}_front_left_caster_hub_wheel_joint" type="continuous">
-       <origin xyz="0.039 0 -0.067" rpy="0 0 0"/>
+       <origin xyz="0.039 0 -0.067" rpy="1.57 0 0"/>
         <parent link="${prefix}_front_left_caster_hub"/>
         <child link="${prefix}_front_left_caster_wheel"/>
-        <axis xyz="0 1 0"/>
-        <dynamics damping="0.5" friction="1.5"/>
-    </joint>
-  <!-- rear-right caster hub -->
+        <axis xyz="0 0 1"/>
+        <dynamics damping="0.5" friction="0.5"/>
+    </joint>
+ <!-- rear-right caster hub -->
     <link name="${prefix}_rear_right_caster_hub">
         <visual>
             <origin xyz="0 0 0" rpy="0 0 0"/>
-            <geometry>
+                <geometry>
+                    <mesh filename="package://amrj16_bin_description/models/meshes/utimac_caster_bin_v1.dae"/>
+                </geometry>
+        </visual>
+    <collision>
+        <origin xyz="0 0 0" rpy="0 0 0"/>
+        <geometry>
                 <mesh filename="package://amrj16_bin_description/models/meshes/utimac_caster_bin_v1.dae"/>
-            </geometry>
-        </visual>
-        <!--collision>
-            <origin xyz="0 0 0" rpy="0 0 0"/>
-            <geometry>
-                <mesh filename="package://amrj16_bin_description/models/meshes/utimac_caster_bin_v1.dae"/>
-            </geometry>
-        </collision -->
-        <inertial>
-            <mass value="1"/>
-            <origin rpy="0 0 0" xyz="0 0 0"/>
-            <inertia ixx="0.0008063" ixy="0.00000393" ixz="-0.00000650" iyy="0.000693" iyz="0.000265" izz="0.0005498"/>
-        </inertial>
+        </geometry>
+    </collision>
+    <inertial>
+        <mass value="0.7"/>
+        <origin rpy="0 0 0" xyz="0 0 0"/>
+        <inertia
+           ixx="0.0008063" ixy="0.00000393" ixz="-0.00000650" iyy="0.000693" iyz="0.000265" izz="0.0005498"/>
+    </inertial>
     </link>
     <joint name="${prefix}_chassis_rear_right_caster_hub_joint" type="continuous">
@@ -207,10 +187,10 @@
         <child link="${prefix}_rear_right_caster_hub"/>
         <axis xyz="0 0 1"/>
-        <dynamics damping="0.5" friction="0.1"/>
-    </joint>
- <!-- rear-right caster wheel -->
-            <link name="${prefix}_rear_right_caster_wheel">
-        <visual>
-            <origin xyz="0 0 0" rpy="1.57 0 0"/>
+        <dynamics damping="0.5" friction="0.5"/>
+    </joint>
+    <!-- rear-right caster wheel -->
+    <link name="${prefix}_rear_right_caster_wheel">
+        <visual>
+            <origin xyz="0 0 0" rpy="0 0 0"/>
                 <geometry>
                     <mesh filename="package://amrj16_bin_description/models/meshes/utimac_wheel_bin_v1.dae"/>
@@ -218,58 +198,48 @@
         </visual>
     <collision>
-        <origin xyz="0 0 0" rpy="1.57  0 0"/>
+        <origin xyz="0 0 0" rpy="0 0 0"/>
         <geometry>
-                <cylinder radius="0.04" length="0.02"/>
+            <cylinder radius="0.040" length="0.02"/>
         </geometry>
     </collision>
     <inertial>
-        <mass value="1"/>
-        <origin rpy="0 0 0" xyz="1.57  0 0"/>
+        <mass value="0.5"/>
+        <origin rpy="0 0 0" xyz="0 0 0"/>
         <inertia
-            ixx="0.0003265" ixy="0" ixz="0" iyy="0.0003265" iyz="0" izz="0.0005849"/>
-    </inertial>
-    </link>
-   <gazebo reference="${prefix}_rear_right_caster_wheel">
-      <collision>
-        <surface>
-          <friction>
-            <ode>
-              <mu>0.3</mu>
-              <mu2>0.3</mu2>
-            </ode>
-            <bullet>
-              <friction>0.3</friction>
-              <friction2>0.3</friction2>
-              <rolling_friction>0.1</rolling_friction>
-            </bullet>
-          </friction>
-        </surface>
-      </collision>
+           ixx="0.0003265" ixy="0" ixz="0" iyy="0.0003265" iyz="0" izz="0.0005849"/>
+    </inertial>
+    </link>
+    <gazebo reference="${prefix}_rear_right_caster_wheel">
+        <kp>5000000000</kp>
+        <kd>5000000000</kd>
+        <mu1>10.0</mu1>
+        <mu2>10.0</mu2>
     </gazebo>
     <joint name="${prefix}_rear_right_caster_hub_wheel_joint" type="continuous">
-       <origin xyz="0.039 0 -0.067" rpy="0 0 0"/>
+       <origin xyz="0.039 0 -0.067" rpy="1.57 0 0"/>
         <parent link="${prefix}_rear_right_caster_hub"/>
         <child link="${prefix}_rear_right_caster_wheel"/>
-        <axis xyz="0 1 0"/>
-        <dynamics damping="0.5" friction="1.5"/>
-    </joint>
-<!-- rear-left caster hub -->
+        <axis xyz="0 0 1"/>
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
File: amrj16_description/urdf/amrj16.xacro (robot description, xacro)
@@ -376,7 +376,24 @@
 </gazebo>
     <link name="asus_xtion">
+        <visual>
+            <origin xyz="0 0 0" rpy="0 0 0"/>
+            <geometry>
+                <mesh filename="package://amrj16_description/models/meshes/amrj16_asus_xtion_pro_live.dae"/>
+            </geometry>
+        </visual>
+            <!--collision>
+                <origin xyz="0 0 0" rpy="0 0 0"/>
+                <geometry>
+                        <cylinder radius="0.030" length="0.041"/>
+                </geometry>
+            </collision-->
+        <inertial>
+            <mass value="0.3"/>
+            <origin rpy="0 0 0" xyz="0 0 0"/>
+            <inertia ixx="0.000025441" ixy="0" ixz="0" iyy="0.00002543" iyz="-0.0000000017817" izz="0.000028616"/>
+        </inertial>
     </link>
     <joint name="chassis_asus_xtion_joint" type="fixed">
-        <origin rpy="0 0 0" xyz="0.300 0.0 0.2"/>
+        <origin rpy="0 0 0" xyz="-0.095 0 0.131"/>
         <parent link="chassis" />
         <child link="asus_xtion" />
