Commit message: Update cartographer options

File: amrj16_description/urdf/amrj16.xacro (robot description, xacro)
@@ -1,6 +1,13 @@
 <?xml version="1.0"?>
     <robot xmlns:xacro="http://www.ros.org/wiki/xacro" name="amrj16">
+    <link name="base_footprint">
+    </link>
     <link name="base_link">
     </link>
+    <joint name="base_link_base_footprintjoint" type="fixed">
+    <origin rpy="0 0 0" xyz="0 0 0.103" />
+    <parent link="base_footprint" />
+    <child link="base_link" />
+  </joint>
     <!-- chassis-->
     <link name="chassis">
@@ -24,5 +31,5 @@
   </link>
   <joint name="base_link_joint" type="fixed">
-    <origin rpy="0 0 0" xyz="0 0 0.0" />
+    <origin rpy="0 0 0" xyz="0 0 0" />
     <parent link="base_link" />
     <child link="chassis" />
@@ -55,5 +62,5 @@
     </gazebo>
     <joint name="chassis_right_wheel_joint" type="continuous">
-        <origin xyz="0 0.5456 0.103" rpy="1.5707 0 0"/>
+        <origin xyz="0 0.5456 0" rpy="1.5707 0 0"/>
         <parent link="chassis"/>
         <child link="right_wheel"/>
@@ -90,5 +97,5 @@
     </gazebo>
     <joint name="chassis_left_wheel_joint" type="continuous">
-        <origin xyz="0 -0.5456 0.103" rpy="1.5707 0 0"/>
+        <origin xyz="0 -0.5456 0" rpy="1.5707 0 0"/>
         <parent link="chassis"/>
         <child link="left_wheel"/>
@@ -119,5 +126,5 @@
     </link>
     <joint name="chassis_front_right_caster_hub_joint" type="continuous">
-        <origin xyz="0.255 0.186 0.053" rpy="0 0 1.5707"/>
+        <origin xyz="0.255 0.186 -0.05" rpy="0 0 1.5707"/>
         <parent link="chassis"/>
         <child link="front_right_caster_hub"/>
@@ -183,5 +190,5 @@
     </link>
     <joint name="chassis_front_left_caster_hub_joint" type="continuous">
-        <origin xyz="0.255 -0.186 0.053" rpy="0 0 1.5707"/>
+        <origin xyz="0.255 -0.186 -0.05" rpy="0 0 1.5707"/>
         <parent link="chassis"/>
         <child link="front_left_caster_hub"/>
@@ -229,5 +236,5 @@
     </link>
     <joint name="camera_dx_joint" type="fixed">
-        <origin rpy="0 0 0" xyz="0.280 0.186 0.068"/>
+        <origin rpy="0 0 0" xyz="0.280 0.186 -0.035"/>
         <parent link="chassis" />
         <child link="rgb_camera_dx" />
@@ -273,5 +280,5 @@
     </link>
     <joint name="rgb_camera_sx_joint" type="fixed">
-        <origin rpy="0 0 0" xyz="0.280 -0.186 0.068"/>
+        <origin rpy="0 0 0" xyz="0.280 -0.186 -0.035"/>
         <parent link="chassis" />
         <child link="rgb_camera_sx" />
@@ -335,5 +342,5 @@
     </link>
     <joint name="chassis_lidar_joint" type="fixed">
-        <origin rpy="0 0 0" xyz="0.200 0 0.0565"/>
+        <origin rpy="0 0 0" xyz="0.200 0 -0.06"/>
         <parent link="chassis" />
         <child link="lidar" />
@@ -431,5 +438,4 @@
       </ros>
       <update_rate>30</update_rate>
-      <joint_name>chassis_forks_joint</joint_name>
       <joint_name>chassis_right_wheel_joint</joint_name>
       <joint_name>chassis_left_wheel_joint</joint_name>
@@ -450,6 +456,6 @@
       <wheel_diameter>0.206</wheel_diameter>
       <!-- limits -->
-      <max_wheel_torque>20.0</max_wheel_torque>
-      <max_wheel_acceleration>2.0</max_wheel_acceleration>
+      <max_wheel_torque>1.0</max_wheel_torque>
+      <max_wheel_acceleration>1.0</max_wheel_acceleration>
       <!--command_topic>cmd_vel</command_topic -->
       <!-- remapping>/cmd_vel:=/cmd_vel</remapping -->
@@ -460,5 +466,5 @@
       <!-- remapping>/odom:=/odom</remapping -->
       <odometry_frame>odom</odometry_frame>
-      <robot_base_frame>base_link</robot_base_frame>
+      <robot_base_frame>base_footprint</robot_base_frame>
     </plugin>
   </gazebo>

Commit message: Add amj16_path_planner_server package

File: amrj16_description/urdf/amrj16.xacro (robot description, xacro)
@@ -430,8 +430,68 @@
         </sensor>
     </gazebo>
+    <link name="imu_link"/>
+    <joint name="imu_joint" type="fixed">
+        <parent link="base_link"/>
+        <child link="imu_link"/>
+        <origin xyz="0.3 0 0" rpy="0 0 0"/>
+    </joint>
+     <gazebo reference="imu_link">
+  <sensor name="br_imu" type="imu">
+    <always_on>true</always_on>
+    <update_rate>100</update_rate>
+    <imu>
+      <angular_velocity>
+        <x>
+          <noise type="gaussian">
+            <mean>0.0</mean>
+            <stddev>2e-4</stddev>
+          </noise>
+        </x>
+        <y>
+          <noise type="gaussian">
+            <mean>0.0</mean>
+            <stddev>2e-4</stddev>
+          </noise>
+        </y>
+        <z>
+          <noise type="gaussian">
+            <mean>0.0</mean>
+            <stddev>2e-4</stddev>
+          </noise>
+        </z>
+      </angular_velocity>
+      <linear_acceleration>
+        <x>
+          <noise type="gaussian">
+            <mean>0.0</mean>
+            <stddev>1.7e-2</stddev>
+          </noise>
+        </x>
+        <y>
+          <noise type="gaussian">
+            <mean>0.0</mean>
+            <stddev>1.7e-2</stddev>
+          </noise>
+        </y>
+        <z>
+          <noise type="gaussian">
+            <mean>0.0</mean>
+            <stddev>1.7e-2</stddev>
+          </noise>
+        </z>
+      </linear_acceleration>
+    </imu>
+    <plugin name="bytes_imu" filename="libgazebo_ros_imu_sensor.so">
+      <ros>
+        <remapping>~/out:=imu</remapping>
+      </ros>
+      <initial_orientation_as_reference>false</initial_orientation_as_reference>
+    </plugin>
+  </sensor>
+</gazebo>
     <!-- PLUGINS -->
-  <!-- JOINT PUBLISHER -->
-  <gazebo>
-    <plugin name="amrj16_joint_state" filename="libgazebo_ros_joint_state_publisher.so">
+    <!-- JOINT PUBLISHER -->
+    <gazebo>
+      <plugin name="amrj16_joint_state" filename="libgazebo_ros_joint_state_publisher.so">
       <ros>
           <remapping>~/out:=joint_states</remapping>

Commit message: Add chassis v.4 repositioning lidar

File: amrj16_description/urdf/amrj16.xacro (robot description, xacro)
@@ -15,5 +15,5 @@
       <origin xyz="0 0 0" rpy="0 0 0"/>
       <geometry>
-        <mesh filename="package://amrj16_description/models/meshes/amrj16_chassis_utimac_v2.dae"/>
+        <mesh filename="package://amrj16_description/models/meshes/amrj16_chassis_utimac_v4.dae"/>
       </geometry>
     </visual>
@@ -21,10 +21,10 @@
       <origin xyz="0 0 0" rpy="0 0 0"/>
       <geometry>
-        <mesh filename="package://amrj16_description/models/meshes/amrj16_chassis_utimac_v2_low_res.stl"/>
+        <mesh filename="package://amrj16_description/models/meshes/amrj16_chassis_utimac_v4_low_res.stl"/>
       </geometry>
     </collision>
     <inertial>
         <mass value="34.2"/>
-        <origin rpy="0 0 0" xyz="0 0 0"/>
+        <origin rpy="0 0 0" xyz="-0.1055 0 -0.0199"/>
         <inertia ixx="10.164712" ixy="0.021460923" ixz="-0.0060724714" iyy="3.4403550" iyz="1.7125796" izz="12.572506"/>
     </inertial>
@@ -126,5 +126,5 @@
     </link>
     <joint name="chassis_front_right_caster_hub_joint" type="continuous">
-        <origin xyz="-0.255 -0.186 -0.05" rpy="0 0 1.5707"/>
+        <origin xyz="-0.255 -0.538 -0.055" rpy="0 0 1.5707"/>
         <parent link="chassis"/>
         <child link="front_right_caster_hub"/>
@@ -154,6 +154,6 @@
     </link>
     <gazebo reference="front_right_caster_wheel">
-        <kp>500</kp>
-        <kd>500</kd>
+        <kp>500000</kp>
+        <kd>500000</kd>
         <mu1>10.0</mu1>
         <mu2>10.0</mu2>
@@ -189,5 +189,5 @@
     </link>
     <joint name="chassis_front_left_caster_hub_joint" type="continuous">
-        <origin xyz="-0.255 0.186 -0.05" rpy="0 0 1.5707"/>
+        <origin xyz="-0.255 0.538 -0.055" rpy="0 0 1.5707"/>
         <parent link="chassis"/>
         <child link="front_left_caster_hub"/>
@@ -217,6 +217,6 @@
     </link>
     <gazebo reference="front_left_caster_wheel">
-        <kp>500</kp>
-        <kd>500</kd>
+        <kp>500000</kp>
+        <kd>500000</kd>
         <mu1>10.0</mu1>
         <mu2>10.0</mu2>
@@ -322,16 +322,16 @@
             <visual>
                 <origin xyz="0 0 0" rpy="0 0 0"/>
-                    <geometry>
-                        <box size="0.02 0.02 0.02"/>
-                    </geometry>
+                <geometry>
+                    <mesh filename="package://amrj16_description/models/meshes/amrj16_rplidarS2.dae"/>
+                </geometry>
             </visual>
-            <collision>
+            <!--collision>
                 <origin xyz="0 0 0" rpy="0 0 0"/>
                 <geometry>
-                        <box size="0.02 0.02 0.02"/>
-                </geometry>
-            </collision>
+                        <cylinder radius="0.030" length="0.041"/>
+                </geometry>
+            </collision-->
             <inertial>
-                <mass value="0.001"/>
+                <mass value="0.3"/>
                 <origin rpy="0 0 0" xyz="0 0 0"/>
                 <inertia
@@ -340,5 +340,5 @@
     </link>
     <joint name="chassis_lidar_joint" type="fixed">
-        <origin rpy="0 0 3.14" xyz="-0.2 0 0.2"/>
+        <origin rpy="3.14 0 0" xyz="-0.2 0 -0.020"/>
         <parent link="chassis" />
         <child link="lidar" />
@@ -347,5 +347,5 @@
 <gazebo reference="lidar">
     <sensor name="sensor_ray" type="ray">
-        <pose>0 0 0 0 0 0</pose> <!-- pose>0 0 0 3.14159265359 0 0</pose -->
+        <pose>0 0 0.040 0 0 0</pose> <!-- pose>0 0 0 3.14159265359 0 0</pose -->
         <ray>
           <scan>
@@ -364,5 +364,5 @@
         <always_on>true</always_on>
         <visualize>true</visualize>
-        <update_rate>40.0</update_rate>
+        <update_rate>50.0</update_rate>
         <plugin name="laser" filename="libgazebo_ros_ray_sensor.so">
           <ros>

Commit message: Add depth camera Realsense D435i

File: amrj16_description/urdf/amrj16.xacro (robot description, xacro)
@@ -445,4 +445,67 @@
         </sensor>
     </gazebo>
+    <!-- new sensor start-->
+    <link name="rgbd_camera_link_frame">
+        <visual>
+        <geometry>
+            <cylinder length="0.01" radius="0.005"/>
+        </geometry>
+        </visual>
+    </link>
+    <joint name="rgbd_camera_link_frame_joint" type="fixed">
+        <origin rpy="0 0 0" xyz="0 0 0"/>
+        <parent link="chassis" />
+        <child link="rgbd_camera_link_frame" />
+        <axis xyz="0 0 0"/>
+    </joint>
+    <link name="camera_depth_frame"/>
+    <joint name="camera_depth_joint" type="fixed">
+      <origin xyz="0 0 0" rpy="0 0 0"/>
+      <parent link="rgbd_camera_link_frame"/>
+      <child link="camera_depth_frame" />
+    </joint>
+    <link name="camera_depth_optical_frame"/>
+    <joint name="camera_depth_optical_joint" type="fixed">
+      <origin xyz="0 0 0" rpy="-1.57 0 -1.57" />
+      <parent link="camera_depth_frame" />
+      <child link="camera_depth_optical_frame" />
+    </joint>
+    <gazebo reference="rgbd_camera_link_frame">
+      <sensor type="depth" name="depth_sensor">
+        <always_on>true</always_on>
+        <update_rate>5.0</update_rate>
+        <camera>
+          <horizontal_fov>${90.0*3.1415926/260.0}</horizontal_fov>
+          <image>
+            <format>R8G8B8</format>
+            <width>640</width>
+            <height>480</height>
+          </image>
+          <clip>
+            <near>0.01</near>
+            <far>2.0</far>
+          </clip>
+        </camera>
+        <plugin name="rgbd_controller" filename="libgazebo_ros_camera.so">
+          <cameraName>amrj16moto</cameraName>
+          <alwaysOn>true</alwaysOn>
+          <updateRate>10</updateRate>
+          <imageTopicName>rgb/image_raw</imageTopicName>
+          <depthImageTopicName>depth/image_raw</depthImageTopicName>
+          <pointCloudTopicName>depth/points</pointCloudTopicName>
+          <cameraInfoTopicName>rgb/camera_info</cameraInfoTopicName>
+          <depthImageCameraInfoTopicName>depth/camera_info</depthImageCameraInfoTopicName>
+          <frame_name>camera_depth_optical_frame</frame_name>
+          <baseline>0.1</baseline>
+          <distortion_k1>0.0</distortion_k1>
+          <distortion_k2>0.0</distortion_k2>
+          <distortion_k3>0.0</distortion_k3>
+          <distortion_t1>0.0</distortion_t1>
+          <distortion_t2>0.0</distortion_t2>
+          <pointCloudCutoff>0.1</pointCloudCutoff>
+        </plugin>
+      </sensor>
+    </gazebo>
+<!-- new sensor end -->
     <link name="imu_link"/>
     <joint name="imu_joint" type="fixed">

Commit message: Updated description and gazebo packages to ROS 2 Humble

File: amrj16_description/urdf/amrj16.xacro (robot description, xacro)
@@ -156,6 +156,6 @@
         <kp>500000</kp>
         <kd>500000</kd>
-        <mu1>10.0</mu1>
-        <mu2>10.0</mu2>
+        <mu1>0.0</mu1>
+        <mu2>0.0</mu2>
     </gazebo>
     <joint name="front_right_caster_hub_wheel_joint" type="continuous">
@@ -219,6 +219,6 @@
         <kp>500000</kp>
         <kd>500000</kd>
-        <mu1>10.0</mu1>
-        <mu2>10.0</mu2>
+        <mu1>0.0</mu1>
+        <mu2>0.0</mu2>
     </gazebo>
     <joint name="front_left_caster_hub_wheel_joint" type="continuous">
@@ -266,5 +266,5 @@
             <update_rate>30</update_rate>
           </camera>
-          <plugin name="camera_controller" filename="libgazebo_ros_camera.so">
+          <plugin name="camera_controller_dx" filename="libgazebo_ros_camera.so">
             <cameraName>rgb_camera</cameraName>
             <imageTopicName>image_raw</imageTopicName>
@@ -310,5 +310,5 @@
             <update_rate>30</update_rate>
           </camera>
-          <plugin name="camera_controller" filename="libgazebo_ros_camera.so">
+          <plugin name="camera_controller_sx" filename="libgazebo_ros_camera.so">
             <cameraName>rgb_camera_sx</cameraName>
             <imageTopicName>image_raw</imageTopicName>
@@ -435,5 +435,5 @@
             <ros>
                 <!-- namespace>/amrj16</namespace -->
-                <argument>~/out:=pointcloud</argument>
+                <remapping>~/out:=pointcloud</remapping>
             </ros>
             <!-- Set output to sensor_msgs/PointCloud to get same output type as gazebo_ros_block_laser -->
@@ -586,5 +586,7 @@
   <!-- Differential drive -->
   <gazebo>
-    <plugin filename="libgazebo_ros_diff_drive.so" name="differential_drive_controller">
+    <plugin name="differential_drive_controller" filename="libgazebo_ros_diff_drive.so">
+      <!-- Update rate -->
+      <update_rate>50</update_rate>
       <!-- wheels -->
       <left_joint>chassis_left_wheel_joint</left_joint>
@@ -594,16 +596,12 @@
       <wheel_diameter>0.206</wheel_diameter>
       <!-- limits -->
-      <max_wheel_torque>20.0</max_wheel_torque>
-      <max_wheel_acceleration>0.3</max_wheel_acceleration>
-      <command_topic>cmd_vel</command_topic>
-      <!-- remapping>/cmd_vel:=/cmd_vel</remapping -->
+      <max_wheel_torque>200.0</max_wheel_torque>
+      <max_wheel_acceleration>2.0</max_wheel_acceleration>
       <!-- output -->
       <publish_odom>true</publish_odom>
       <publish_odom_tf>true</publish_odom_tf>
-      <odometry_topic>odom</odometry_topic>
-      <!-- remapping>/odom:=/odom</remapping -->
+      <publish_wheel_tf>false</publish_wheel_tf>
       <odometry_frame>odom</odometry_frame>
       <robot_base_frame>base_footprint</robot_base_frame>
-      <!--odometry_source>1</odometry_source -->
     </plugin>
   </gazebo>
@@ -629,3 +627,4 @@
     </plugin>
   </gazebo> -->
+  <xacro:include filename="$(find amrj16_description)/urdf/amrj16_plugins.xacro" />
 </robot>

File: amrj16_description/urdf/amrj16_plugins.xacro (robot description, xacro)
@@ -1,69 +1,4 @@
 <?xml version="1.0"?>
 <robot xmlns:xacro="http://www.ros.org/wiki/xacro" name="amrj16">
-    <!-- PLUGINS -->
-  <!-- JOINT PUBLISHER -->
-  <gazebo>
-    <plugin name="amrj16_joint_state" filename="libgazebo_ros_joint_state_publisher.so">
-      <ros>
-          <remapping>~/out:=joint_states</remapping>
-      </ros>
-      <update_rate>30</update_rate>
-      <joint_name>chassis_forks_joint</joint_name>
-      <joint_name>chassis_right_wheel_joint</joint_name>
-      <joint_name>chassis_left_wheel_joint</joint_name>
-      <joint_name>chassis_front_right_caster_hub_joint</joint_name>
-      <joint_name>front_right_caster_hub_wheel_joint</joint_name>
-      <joint_name>chassis_rear_right_caster_hub_joint</joint_name>
-      <joint_name>rear_right_caster_hub_wheel_joint</joint_name>
-      <joint_name>chassis_front_left_caster_hub_joint</joint_name>
-      <joint_name>front_left_caster_hub_wheel_joint</joint_name>
-      <joint_name>chassis_rear_left_caster_hub_joint</joint_name>
-      <joint_name>rear_left_caster_hub_wheel_joint</joint_name>
-    </plugin>
-  </gazebo>
-  <!-- Differential drive -->
-  <gazebo>
-    <plugin filename="libgazebo_ros_diff_drive.so" name="differential_drive_controller">
-      <!-- wheels -->
-      <left_joint>chassis_left_wheel_joint</left_joint>
-      <right_joint>chassis_right_wheel_joint</right_joint>
-      <!-- kinematics -->
-      <wheel_separation>1.0912</wheel_separation>
-      <wheel_diameter>0.206</wheel_diameter>
-      <!-- limits -->
-      <max_wheel_torque>20.0</max_wheel_torque>
-      <max_wheel_acceleration>2.0</max_wheel_acceleration>
-      <command_topic>cmd_vel</command_topic>
-      <remapping>/cmd_vel:=${ns}/cmd_vel</remapping>
-      <!-- output -->
-      <publish_odom>true</publish_odom>
-      <publish_odom_tf>true</publish_odom_tf>
-      <publish_wheel_tf>false</publish_wheel_tf>
-      <odometry_topic>odom</odometry_topic>
-      <remapping>/odom:=${ns}/odom</remapping>
-      <odometry_frame>odom</odometry_frame>
-      <robot_base_frame>base_link</robot_base_frame>
-    </plugin>
-  </gazebo>
-    <!-- Position Config -->
-  <ros2_control name="GazeboSystem" type="system">
-      <hardware>
-        <plugin>gazebo_ros2_control/GazeboSystem</plugin>
-      </hardware>
-      <joint name="chassis_forks_joint">
-        <command_interface name="position">
-          <param name="min">0</param>
-          <param name="max">0.035</param>
-        </command_interface>
-        <state_interface name="position"/>
-        <state_interface name="velocity"/>
-        <state_interface name="effort"/>
-      </joint>
-  </ros2_control>
-  <gazebo>
-    <plugin filename="libgazebo_ros2_control.so" name="gazebo_ros2_control">
-      <parameters>$(find amrj16_description)/config/amrj16_controller_position.yaml</parameters>
-      <robot_param_node>robot_state_publisher_node</robot_param_node>
-    </plugin>
-  </gazebo>
+    <!-- Plugins are currently inside amrj16.xacro, so this file is left empty to prevent duplication and crashes. -->
 </robot>
